Commit message: Revision of joint names, links, rotating tilt_joint

File: crom2_description/robots/crom2.urdf.xacro (robot description, xacro)
@@ -17,27 +17,15 @@
    <xacro:include filename="$(find crom2_description)/urdf/crom2_head.urdf.xacro" />
    <!--xacro:include filename="$(find crom2_description)/urdf/crom2_head.urdf.xacro" /-->
+  <link name="base_footprint">
+  </link>
    <!-- Add the base -->
-   <base name="base" color="Blue"/>
+   <base name="base" color="Blue" parent="base_footprint"/>
    <!-- Attach the trunk -->
-   <trunk name="trunk" parent="base" color="Blue">
+   <trunk name="waist" parent="base" color="Blue">
       <origin xyz="${trunk_offset_x} ${trunk_offset_y} ${trunk_offset_z}" rpy="0 0 0" />
    </trunk>
    <!-- Attach the head -->
-   <head name="head" parent="trunk" color="Blue">
+   <head name="head" parent="waist" color="Blue">
       <origin xyz="${head_offset_x} ${head_offset_y} ${head_offset_z}" rpy="0 0 0" />
    </head>
-  <link name="base_footprint">
-      <visual>
-        <origin xyz="0 0 0" rpy="0 0 0" />
-        <geometry>
-          <box size="0.05 0.05 0.01" />
-        </geometry>
-        <!--material name="TransparentGreen" /-->
-      </visual>
-  </link>
-  <joint name="$base_joint" type="fixed">
-    <origin xyz="0 0 0" rpy="0 0 0" />
-    <parent link="base_footprint"/>
-    <child link="base_link" />
-  </joint>
 </robot>

File: crom2_description/urdf/crom2_base.urdf.xacro (robot description, xacro)
@@ -8,5 +8,5 @@
   <property name="PI" value="3.1415" />
   <!-- The base xacro macro -->
-  <macro name="base" params="name color">
+  <macro name="base" params="name parent color">
     <link name="${name}_link">
       <visual>
@@ -24,4 +24,9 @@
       </collision>
     </link>
+    <joint name="${name}_joint" type="fixed">
+		<origin xyz="0 0 0" rpy="0 0 0" />
+		<parent link="${parent}"/>
+		<child link="${name}_link" />
+	</joint>
   </macro>
  </robot>

File: crom2_description/urdf/crom2_head.urdf.xacro (robot description, xacro)
@@ -9,10 +9,10 @@
   <!-- Define the head -->
   <macro name="head" params="parent name color *origin">
-	<joint name="${parent}_${name}_joint" type="fixed">
+	<joint name="${name}_frame_joint" type="fixed">
       <xacro:insert_block name="origin" />
       <parent link="${parent}_link"/>
-      <child link="${name}_pan_tilt_1_link"/>
+      <child link="${name}_frame_link"/>
     </joint>
-    <link name="${name}_pan_tilt_1_link">
+    <link name="${name}_frame_link">
       <visual>
         <origin xyz="0 0 0" rpy="0 0 0" />
@@ -29,10 +29,10 @@
       </collision>
     </link>
-    <joint name="${name}_pan-tilt_2_joint" type="fixed">
+    <joint name="${name}_pan_motor_joint" type="fixed">
       <origin xyz="0 0 0" rpy="0 0 0" />
-      <parent link="${name}_pan_tilt_1_link"/>
-      <child link="${name}_dynamixel_L42_pan_link"/>
+      <parent link="${name}_frame_link"/>
+      <child link="${name}_pan_motor_link"/>
     </joint>
-    <link name="${name}_dynamixel_L42_pan_link">
+    <link name="${name}_pan_motor_link">
       <visual>
         <origin xyz="0 0 0" rpy="0 0 0" />
@@ -51,10 +51,10 @@
     <joint name="${name}_pan_joint" type="revolute">
       <origin xyz="0 0 0.111" rpy="0 0 0" />
-      <parent link="${name}_dynamixel_L42_pan_link"/>
-      <child link="${name}_pan_tilt_2_link"/>
+      <parent link="${name}_pan_motor_link"/>
+      <child link="${name}_pan_link"/>
       <axis xyz="0 0 1" />
 	  <limit effort="1.5" velocity="6.178465545" lower="-1.58" upper="1.58" />
     </joint>
-    <link name="${name}_pan_tilt_2_link">
+    <link name="${name}_pan_link">
       <visual>
         <origin xyz="0 0 0" rpy="0 0 0" />
@@ -72,13 +72,13 @@
     </link>
     <joint name="${name}_tilt_joint" type="revolute">
-      <origin xyz="0 0 0" rpy="0 0 0" />
-      <parent link="${name}_pan_tilt_2_link"/>
-      <child link="${name}_dynamixel_L42_tilt_link"/>
-      <axis xyz="0 1 0" />
-	  <limit effort="1.5" velocity="6.178465545" lower="-1.58" upper="1.58" />
+      <origin xyz="0 0 0" rpy="-1.57079 0 0" />
+      <parent link="${name}_pan_link"/>
+      <child link="${name}_tilt_link"/>
+      <axis xyz="0 0 1" />
+	  <limit effort="1.5" velocity="6.178465545" lower="-1.57079" upper="1.57079" />
     </joint>
-    <link name="${name}_dynamixel_L42_tilt_link">
-      <visual>
-        <origin xyz="0 -0.027 0" rpy="-1.58 0 0" />
+    <link name="${name}_tilt_link">
+		<visual>
+        <origin xyz="0 0 -0.027" rpy="0 0 0" />
         <geometry>
           <mesh filename = "package://crom2_description/meshes/dynamixel_L42.STL" />
@@ -87,5 +87,5 @@
       </visual>
       <collision>
-        <origin xyz="0 -0.027 0" rpy="-1.58 0 0" />
+        <origin xyz="0 0 -0.027" rpy="0 0 0" />
         <geometry>
           <mesh filename = "package://crom2_description/meshes/dynamixel_L42.STL" />
@@ -93,10 +93,10 @@
       </collision>
     </link>
-    <joint name="${name}_pan_tilt_3_joint" type="fixed">
+    <joint name="${name}_tilt_motor_2_joint" type="fixed">
       <origin xyz="0 0 0" rpy="0 0 0" />
-      <parent link="${name}_dynamixel_L42_tilt_link"/>
-      <child link="${name}_pan_tilt_3_link"/>
+      <parent link="${name}_pan_link"/>
+      <child link="${name}_tilt_aux_link"/>
     </joint>
-    <link name="${name}_pan_tilt_3_link">
+    <link name="${name}_tilt_aux_link">
       <visual>
         <origin xyz="0 -0.027 0" rpy="0 0 0" />
@@ -113,10 +113,10 @@
       </collision>
     </link>
-    <joint name="${name}_pan_tilt_4_joint" type="fixed">
-      <origin xyz="0 0 0.021" rpy="0 0 0" />
-      <parent link="${name}_dynamixel_L42_tilt_link"/>
-      <child link="${name}_pan_tilt_4_link"/>
+    <joint name="${name}_camera_frame_joint" type="fixed">
+      <origin xyz="0 -0.021 0" rpy="1.57079  0 0" />
+      <parent link="${name}_tilt_link"/>
+      <child link="${name}_camera_frame_link"/>
     </joint>
-    <link name="${name}_pan_tilt_4_link">
+    <link name="${name}_camera_frame_link">
       <visual>
         <origin xyz="0 0 0" rpy="0 0 0" />
@@ -135,5 +135,5 @@
     <joint name="${name}_f10_camera_right_joint" type="fixed">
       <origin xyz="0.0075 -0.055 0.015" rpy="0 0 0" />
-      <parent link="${name}_pan_tilt_4_link"/>
+      <parent link="${name}_camera_frame_link"/>
       <child link="${name}_f10_camera_right_link"/>
     </joint>
@@ -155,5 +155,5 @@
       <joint name="${name}_f10_camera_left_joint" type="fixed">
       <origin xyz="0.0075 0.055 0.015" rpy="0 0 0" />
-      <parent link="${name}_pan_tilt_4_link"/>
+      <parent link="${name}_camera_frame_link"/>
       <child link="${name}_f10_camera_left_link"/>
     </joint>
@@ -175,5 +175,5 @@
     <joint name="${name}_xtion_camera_joint" type="fixed">
       <origin xyz="0.041 0 0.065" rpy="0 0 0" />
-      <parent link="${name}_pan_tilt_4_link"/>
+      <parent link="${name}_camera_frame_link"/>
       <child link="${name}_xtion_camera_link"/>
     </joint>

File: crom2_description/urdf/crom2_trunk.urdf.xacro (robot description, xacro)
@@ -1,3 +1,3 @@
-<?x	ml version="1.0"?>
+<?xml version="1.0"?>
 <robot name="trunk" xmlns:xacro="http://ros.org/wiki/xacro">
   <!-- Define a number of dimensions using properties -->
@@ -8,11 +8,11 @@
   <!-- Define the torso -->
   <macro name="trunk" params="parent name color *origin">
-    <joint name="waist_joint" type="revolute">
-			<xacro:insert_block name="origin" />
-			<parent link="${parent}_link" />
-			<child link="${name}_link" />
-			<axis xyz="0 0 1" />
-			<limit effort="1.5" velocity="6.178465545" lower="-1.58" upper="1.58" />
-		</joint>
+    <joint name="${name}_joint" type="revolute">
+		<xacro:insert_block name="origin" />
+		<parent link="${parent}_link" />
+		<child link="${name}_link" />
+		<axis xyz="0 0 1" />
+		<limit effort="1.5" velocity="6.178465545" lower="-1.58" upper="1.58" />
+	</joint>
 	<link name="${name}_link">
       <visual>
