Commit message: modifications and gazebo specifications

File: crom2_description/robots/crom2.gazebo.xacro (robot description, xacro)
@@ -1,101 +1,12 @@
 <?xml version="1.0"?>
 <robot xmlns:xacro="http://ros.org/wiki/xacro">
-  <gazebo>
-	<plugin name="gazebo_ros_control" filename="libgazebo_ros_control.so">
-		<robotNamespace>/crom</robotNamespace>
-		<controlPeriod>0.001</controlPeriod>
-		<robotSimType>gazebo_ros_control/DefaultRobotHWSim</robotSimType>
-	</plugin>
-  </gazebo>
-  <gazebo reference="base_link">
-    <material>Gazebo/FlatBlack</material>
-    <turnGravityOff>false</turnGravityOff>
-    <selfCollide>true</selfCollide>
-  </gazebo>
-  <gazebo reference="waist_link">
-    <material>Gazebo/Blue</material>
-    <turnGravityOff>false</turnGravityOff>
-    <selfCollide>true</selfCollide>
-  </gazebo>
-  <!--Cameras-->
-  <!-- camera_2_hand_left_link -->
-  <gazebo reference="camera_2_hand_left_link">
-    <sensor type="camera" name="camera_hand_left">
-      <update_rate>30.0</update_rate>
-      <camera name="camera_hand_left">
-        <horizontal_fov>1.3962634</horizontal_fov>
-        <image>
-          <width>800</width>
-          <height>800</height>
-          <format>R8G8B8</format>
-        </image>
-        <clip>
-          <near>0.02</near>
-          <far>300</far>
-        </clip>
-        <noise>
-          <type>gaussian</type>
-          <!-- Noise is sampled independently per pixel on each frame.
-               That pixel's noise value is added to each of its color
-               channels, which at that point lie in the range [0,1]. -->
-          <mean>0.0</mean>
-          <stddev>0.007</stddev>
-        </noise>
-      </camera>
-      <plugin name="camera_controller" filename="libgazebo_ros_camera.so">
-        <alwaysOn>true</alwaysOn>
-        <updateRate>0.0</updateRate>
-        <cameraName>crom/camera_hand_left</cameraName>
-        <imageTopicName>image_raw</imageTopicName>
-        <cameraInfoTopicName>camera_hand_left_info</cameraInfoTopicName>
-        <frameName>camera_2_hand_left_link</frameName>
-        <hackBaseline>0.07</hackBaseline>
-        <distortionK1>0.0</distortionK1>
-        <distortionK2>0.0</distortionK2>
-        <distortionK3>0.0</distortionK3>
-        <distortionT1>0.0</distortionT1>
-        <distortionT2>0.0</distortionT2>
-      </plugin>
-    </sensor>
-  </gazebo>
-    <!-- camera_2_hand_right_link -->
-  <gazebo reference="camera_2_hand_right_link">
-    <sensor type="camera" name="camera_hand_right">
-      <update_rate>30.0</update_rate>
-      <camera name="camera_hand_right">
-        <horizontal_fov>1.3962634</horizontal_fov>
-        <image>
-          <width>800</width>
-          <height>800</height>
-          <format>R8G8B8</format>
-        </image>
-        <clip>
-          <near>0.02</near>
-          <far>300</far>
-        </clip>
-        <noise>
-          <type>gaussian</type>
-          <!-- Noise is sampled independently per pixel on each frame.
-               That pixel's noise value is added to each of its color
-               channels, which at that point lie in the range [0,1]. -->
-          <mean>0.0</mean>
-          <stddev>0.007</stddev>
-        </noise>
-      </camera>
-      <plugin name="camera_controller" filename="libgazebo_ros_camera.so">
-        <alwaysOn>true</alwaysOn>
-        <updateRate>0.0</updateRate>
-        <cameraName>crom/camera_hand_right</cameraName>
-        <imageTopicName>image_raw</imageTopicName>
-        <cameraInfoTopicName>camera_hand_right_info</cameraInfoTopicName>
-        <frameName>camera_2_hand_right_link</frameName>
-        <hackBaseline>0.07</hackBaseline>
-        <distortionK1>0.0</distortionK1>
-        <distortionK2>0.0</distortionK2>
-        <distortionK3>0.0</distortionK3>
-        <distortionT1>0.0</distortionT1>
-        <distortionT2>0.0</distortionT2>
-      </plugin>
-    </sensor>
-  </gazebo>
+  <xacro:macro name="crom2_gazebo">
+	  <gazebo>
+		<plugin name="gazebo_ros_control" filename="libgazebo_ros_control.so">
+			<robotNamespace>/crom2</robotNamespace>
+			<controlPeriod>0.001</controlPeriod>
+			<robotSimType>gazebo_ros_control/DefaultRobotHWSim</robotSimType>
+		</plugin>
+	  </gazebo>
+  </xacro:macro>
 </robot>

File: crom2_description/robots/crom2_no_arms.urdf.xacro (robot description, xacro)
@@ -1,8 +1,17 @@
 <?xml version="1.0"?>
 <robot name="crom2_robot" xmlns:xacro="http://ros.org/wiki/xacro">
+	<!-- Include all component files -->
+   <xacro:include filename="$(find crom2_description)/urdf/material/materials.urdf.xacro" />
+   <xacro:include filename="$(find crom2_description)/urdf/model/crom2_base.urdf.xacro" />
+   <xacro:include filename="$(find crom2_description)/urdf/model/crom2_trunk.urdf.xacro" />
+   <xacro:include filename="$(find crom2_description)/urdf/model/crom2_head.urdf.xacro" />
+   <xacro:include filename="$(find crom2_description)/robots/crom2.gazebo.xacro" />
+   <!--xacro:include filename="$(find crom2_description)/urdf/crom2_head.urdf.xacro" /-->
    <!-- Define a offsets using properties -->
-   <property name="torso_offset_x" value="0.0" />
-   <property name="torso_offset_y" value="0.0" />
-   <property name="torso_offset_z" value="0.0" />
+   <property name="reverse" value="-1.0" />
+   <property name="M_PI" value="3.1415926535897931" />
+   <property name="base_offset_x" value="0.0" />
+   <property name="base_offset_y" value="0.0" />
+   <property name="base_offset_z" value="0.0" />
    <property name="trunk_offset_x" value="0.0" />
    <property name="trunk_offset_y" value="0.0" />
@@ -11,21 +20,18 @@
    <property name="head_offset_y" value="0.0" />
    <property name="head_offset_z" value="0.545" />
-   <!-- Include all component files -->
-   <xacro:include filename="$(find crom2_description)/urdf/material/materials.urdf.xacro" />
-   <xacro:include filename="$(find crom2_description)/urdf/model/crom2_base.urdf.xacro" />
-   <xacro:include filename="$(find crom2_description)/urdf/model/crom2_trunk.urdf.xacro" />
-   <xacro:include filename="$(find crom2_description)/urdf/model/crom2_head.urdf.xacro" />
-   <!--xacro:include filename="$(find crom2_description)/urdf/crom2_head.urdf.xacro" /-->
   <link name="base_footprint">
   </link>
    <!-- Add the base -->
-   <base name="base" parent="base_footprint" color="Blue"/>
+   <base_model name="base" parent="base_footprint" color="Blue">
+   </base_model>
    <!-- Attach the trunk -->
-   <trunk name="waist" parent="base" color="Blue">
+   <trunk_model name="waist" parent="base" color="Blue">
       <origin xyz="${trunk_offset_x} ${trunk_offset_y} ${trunk_offset_z}" rpy="0 0 0" />
-   </trunk>
+   </trunk_model>
    <!-- Attach the head -->
-   <head name="head" parent="waist" color="Blue">
+   <head_model name="head" parent="waist" color="Blue">
       <origin xyz="${head_offset_x} ${head_offset_y} ${head_offset_z}" rpy="0 0 0" />
-   </head>
+   </head_model>
+   <!--Add robot gazebo macro -->
+   <crom2_gazebo />
 </robot>

File: crom2_description/urdf/gazebo/crom2_head.gazebo.xacro (robot description, xacro)
@@ -2,9 +2,13 @@
 <robot xmlns:xacro="http://ros.org/wiki/xacro">
 	<xacro:macro name="head_gazebo" params="name">
-		<gazebo reference="${name}_start_link">
+		<gazebo reference="$${name}_base_link">
 			<fdir1 value="1 0 0"/>
 			<maxVel>2.0</maxVel>
 			<material>Gazebo/Grey</material>
 			<turnGravityOff>false</turnGravityOff>
+		</gazebo>
+		<gazebo reference="${name}_pan_motor_link">
+			<fdir1 value="1 0 0"/>
+			<maxVel>2.0</maxVel>
 		</gazebo>
 		<gazebo reference="${name}_pan_link">
@@ -14,18 +18,22 @@
 			<turnGravityOff>false</turnGravityOff>
 		</gazebo>
+		<gazebo reference="${name}_tilt_motor_link">
+			<fdir1 value="1 0 0"/>
+			<maxVel>2.0</maxVel>
+		</gazebo>
 		<gazebo reference="${name}_tilt_link">
 			<fdir1 value="1 0 0"/>
-			<maxVel>2.0</maxVel>
+			<material>Gazebo/FlatBlack</material>
 			<material>Gazebo/Grey</material>
 			<turnGravityOff>false</turnGravityOff>
 		</gazebo>
-		<gazebo reference="${name}_camera_structure_link">
+		<gazebo reference="${name}_camera_frame">
 			<material>Gazebo/FlatBlack</material>
 		</gazebo>
-	   <!-- camera_head_left_link -->
-	  <gazebo reference="${name}_camera_left_link">
-		<sensor type="camera" name="camera_head_left">
+	  <!-- camera_head_left_link -->
+	  <gazebo reference="${name}_f10_camera_left_optical_frame">
+		<sensor type="camera" name="${name}_f10_camera_left">
 		  <update_rate>30.0</update_rate>
-		  <camera name="camera_head_left">
+		  <camera name="${name}_f10_camera_left">
 			<horizontal_fov>1.3962634</horizontal_fov>
 			<image>
@@ -63,9 +71,9 @@
 		</sensor>
 	  </gazebo>
-		<!-- camera_head_right_link -->
-	  <gazebo reference="${name}_camera_right_link">
-		<sensor type="camera" name="camera_head_right">
+	  <!-- camera_head_right_link -->
+	  <gazebo reference="{name}_f10_camera_right_optical_frame">
+		<sensor type="camera" name="${name}_f10_camera_right">
 		  <update_rate>30.0</update_rate>
-		  <camera name="camera_head_right">
+		  <camera name="${name}_f10_camera_right">
 			<horizontal_fov>1.3962634</horizontal_fov>
 			<image>

File: crom2_description/urdf/model/crom2_base.urdf.xacro (robot description, xacro)
@@ -1,13 +1,17 @@
 <?xml version="1.0"?>
 <robot name="base" xmlns:xacro="http://ros.org/wiki/xacro">
+  <xacro:include filename="$(find crom2_description)/urdf/gazebo/crom2_base.gazebo.xacro" />
   <!-- Define a number of dimensions using properties -->
   <property name="base_size_x" value="0.55" />
   <property name="base_size_y" value="0.55" />
   <property name="base_size_z" value="1.078" />
-  <property name="mesh_scale" value="1" />
-  <property name="PI" value="3.1415" />
   <!-- The base xacro macro -->
-  <macro name="base" params="name parent color">
-    <link name="${name}_link">
+  <xacro:macro name="base_model" params="name parent color">
+    <joint name="${name}_joint" type="fixed">
+		<origin xyz="0 0 0" rpy="0 0 0" />
+		<parent link="${parent}"/>
+		<child link="${name}_link" />
+	</joint>
+	<link name="${name}_link">
       <visual>
         <origin xyz="0 0 0" rpy="0 0 0" />
@@ -20,14 +24,10 @@
         <origin xyz="0 0 0" rpy="0 0 0" />
         <geometry>
-          <!--box size="${base_size_x} ${base_size_y} ${base_size_z}" /-->
-           <mesh filename = "package://crom2_description/meshes/CROM2_base.dae"/>
+          <mesh filename = "package://crom2_description/meshes/CROM2_base.dae"/>
         </geometry>
       </collision>
     </link>
-    <joint name="${name}_joint" type="fixed">
-		<origin xyz="0 0 0" rpy="0 0 0" />
-		<parent link="${parent}"/>
-		<child link="${name}_link" />
-	</joint>
-  </macro>
+	<!--Add base_gazebo macro -->
+	<base_gazebo name="${name}" />
+  </xacro:macro>
  </robot>
