Commit message: modifications and gazebo specifications

File: crom2_description/urdf/model/crom2_head.urdf.xacro (robot description, xacro)
@@ -1,211 +1,251 @@
 <?xml version="1.0"?>
 <robot name="head" xmlns:xacro="http://ros.org/wiki/xacro">
-  <!-- Define a number of dimensions using properties -->
-  <property name="head_pan_offset_x" value="0.45" />
-  <property name="head_pan_offset_y" value="0.45" />
-  <property name="head_size_y" value="0.284" />
-  <property name="head_size_z" value="0.545" />
-  <property name="mesh_scale" value="1" />
-  <property name="M_PI" value="3.1415926535897931" />
-  <!-- Define the head -->
-  <macro name="head" params="parent name color *origin">
-	<joint name="${name}_frame_joint" type="fixed">
-      <xacro:insert_block name="origin" />
-      <parent link="${parent}_link"/>
-      <child link="${name}_frame_link"/>
-    </joint>
-    <link name="${name}_frame_link">
-      <visual>
-        <origin xyz="0 0 0" rpy="0 0 0" />
-        <geometry>
-          <mesh filename = "package://crom2_description/meshes/CROM2_pantilt_1.STL"/>
-        </geometry>
-        <material name="Blue" />
-      </visual>
-      <collision>
-        <origin xyz="0 0 0" rpy="0 0 0" />
-        <geometry>
-          <mesh filename = "package://crom2_description/meshes/CROM2_pantilt_1.dae" />
-        </geometry>
-      </collision>
-    </link>
-    <joint name="${name}_pan_motor_joint" type="fixed">
-      <origin xyz="0 0 0" rpy="0 0 0" />
-      <parent link="${name}_frame_link"/>
-      <child link="${name}_pan_motor_link"/>
-    </joint>
-    <link name="${name}_pan_motor_link">
-      <visual>
-        <origin xyz="0 0 0" rpy="0 0 0" />
-        <geometry>
-          <mesh filename = "package://crom2_description/meshes/dynamixel_L42.STL" />
-        </geometry>
-        <material name="Black" />
-      </visual>
-      <collision>
-        <origin xyz="0 0 0" rpy="0 0 0" />
-        <geometry>
-          <mesh filename = "package://crom2_description/meshes/dynamixel_L42.dae" />
-        </geometry>
-      </collision>
-    </link>
-    <joint name="${name}_pan_joint" type="revolute">
-      <origin xyz="0 0 0.111" rpy="0 0 0" />
-      <parent link="${name}_pan_motor_link"/>
-      <child link="${name}_pan_link"/>
-      <axis xyz="0 0 1" />
-	  <limit effort="1.5" velocity="6.178465545" lower="-1.58" upper="1.58" />
-    </joint>
-    <link name="${name}_pan_link">
-      <visual>
-        <origin xyz="0 0 0" rpy="0 0 0" />
-        <geometry>
-          <mesh filename = "package://crom2_description/meshes/CROM2_pantilt_2.STL" />
-        </geometry>
-        <material name="Blue" />
-      </visual>
-      <collision>
-        <origin xyz="0 0 0" rpy="0 0 0" />
-        <geometry>
-          <mesh filename = "package://crom2_description/meshes/CROM2_pantilt_2.dae" />
-        </geometry>
-      </collision>
-    </link>
-    <joint name="${name}_tilt_joint" type="revolute">
-      <origin xyz="0 0 0" rpy="-1.57079 0 0" />
-      <parent link="${name}_pan_link"/>
-      <child link="${name}_tilt_link"/>
-      <axis xyz="0 0 -1" />
-	  <limit effort="1.5" velocity="6.178465545" lower="-1.57079" upper="1.57079" />
-    </joint>
-    <link name="${name}_tilt_link">
-		<visual>
-        <origin xyz="0 0 -0.027" rpy="0 0 0" />
-        <geometry>
-          <mesh filename = "package://crom2_description/meshes/dynamixel_L42.STL" />
-        </geometry>
-        <material name="Black" />
-      </visual>
-      <collision>
-        <origin xyz="0 0 -0.027" rpy="0 0 0" />
-        <geometry>
-          <mesh filename = "package://crom2_description/meshes/dynamixel_L42.dae" />
-        </geometry>
-      </collision>
-    </link>
-    <joint name="${name}_tilt_motor_2_joint" type="fixed">
-      <origin xyz="0 0 0" rpy="0 0 0" />
-      <parent link="${name}_pan_link"/>
-      <child link="${name}_tilt_aux_link"/>
-    </joint>
-    <link name="${name}_tilt_aux_link">
-      <visual>
-        <origin xyz="0 -0.027 0" rpy="0 0 0" />
-        <geometry>
-          <mesh filename = "package://crom2_description/meshes/CROM2_pantilt_3.STL" />
-        </geometry>
-        <material name="Grey" />
-      </visual>
-      <collision>
-        <origin xyz="0 -0.027 0" rpy="0 0 0" />
-        <geometry>
-          <mesh filename = "package://crom2_description/meshes/CROM2_pantilt_3.dae" />
-        </geometry>
-      </collision>
-    </link>
-    <joint name="${name}_camera_frame_joint" type="fixed">
-      <origin xyz="0 -0.021 0" rpy="1.57079  0 0" />
-      <parent link="${name}_tilt_link"/>
-      <child link="${name}_camera_frame"/>
-    </joint>
-    <link name="${name}_camera_frame">
-      <visual>
-        <origin xyz="0 0 0" rpy="0 0 0" />
-        <geometry>
-          <mesh filename = "package://crom2_description/meshes/CROM2_pantilt_4.STL" />
-        </geometry>
-        <material name="Blue" />
-      </visual>
-      <collision>
-        <origin xyz="0 0 0" rpy="0 0 0" />
-        <geometry>
-          <mesh filename = "package://crom2_description/meshes/CROM2_pantilt_4.dae" />
-        </geometry>
-      </collision>
-    </link>
-    <joint name="${name}_f10_camera_right_joint" type="fixed">
-      <origin xyz="0.0075 -0.055 0.015" rpy="0 0 0" />
-      <parent link="${name}_camera_frame"/>
-      <child link="${name}_f10_camera_right_frame"/>
-    </joint>
-    <link name="${name}_f10_camera_right_frame">
-      <visual>
-        <origin xyz="0 0 0" rpy="0 0 0" />
-        <geometry>
-          <mesh filename = "package://crom2_description/meshes/FL2-010-R0-camera.STL" />
-        </geometry>
-        <material name="Black" />
-      </visual>
-      <collision>
-        <origin xyz="0 0 0" rpy="0 0 0" />
-        <geometry>
-          <mesh filename = "package://crom2_description/meshes/FL2-010-R0-camera.dae" />
-        </geometry>
-      </collision>
-    </link>
-    <joint name="${name}_f10_camera_right_optical_joint" type="fixed">
-      <origin xyz="0.0 0.0 0.0145" rpy="${M_PI/2} 0 ${M_PI/2}" />
-      <parent link="${name}_f10_camera_right_frame"/>
-      <child link="${name}_f10_camera_right_optical_frame"/>
-    </joint>
-    <link name="${name}_f10_camera_right_optical_frame">
-    </link>
-    <joint name="${name}_f10_camera_left_joint" type="fixed">
-      <origin xyz="0.0075 0.055 0.015" rpy="0 0 0" />
-      <parent link="${name}_camera_frame"/>
-      <child link="${name}_f10_camera_left_frame"/>
-    </joint>
-    <link name="${name}_f10_camera_left_frame">
-      <visual>
-        <origin xyz="0 0 0" rpy="0 0 0" />
-        <geometry>
-          <mesh filename = "package://crom2_description/meshes/FL2-010-R0-camera.STL" />
-        </geometry>
-        <material name="Black" />
-      </visual>
-      <collision>
-        <origin xyz="0 0 0" rpy="0 0 0" />
-        <geometry>
-          <mesh filename = "package://crom2_description/meshes/FL2-010-R0-camera.dae" />
-        </geometry>
-      </collision>
-    </link>
-    <joint name="${name}_f10_camera_left_optical_joint" type="fixed">
-      <origin xyz="0.0 0.0 0.0145" rpy="${M_PI/2} 0 ${M_PI/2}" />
-      <parent link="${name}_f10_camera_left_frame"/>
-      <child link="${name}_f10_camera_left_optical_frame"/>
-    </joint>
-    <link name="${name}_f10_camera_left_optical_frame">
-    </link>
-    <joint name="${name}_xtion_camera_joint" type="fixed">
-      <origin xyz="0.041 0 0.065" rpy="0 0 0" />
-      <parent link="${name}_camera_frame"/>
-      <child link="${name}_xtion_camera_frame"/>
-    </joint>
-    <link name="${name}_xtion_camera_frame">
-      <visual>
-        <origin xyz="0 0 0" rpy="0 0 0" />
-        <geometry>
-          <mesh filename = "package://crom2_description/meshes/xtion_camera.STL" />
-        </geometry>
-        <material name="Black" />
-      </visual>
-      <collision>
-        <origin xyz="0 0 0" rpy="0 0 0" />
-        <geometry>
-          <mesh filename = "package://crom2_description/meshes/xtion_camera.dae" />
-        </geometry>
-      </collision>
-    </link>
-  </macro>
+	<xacro:include filename="$(find crom2_description)/urdf/gazebo/crom2_head.gazebo.xacro" />
+	<!--xacro:include filename="$(find crom2_description)/urdf/transmission/crom2_head.transmission.xacro" /-->
+	<!-- Define a number of dimensions using properties -->
+	<xacro:property name="head_pan_joint_offset_z" value="0.111" />
+	<xacro:property name="head_tilt_servo_offset" value="0.027" />
+	<xacro:property name="head_size_x" value="0.188" />
+	<xacro:property name="head_size_y" value="0.180" />
+	<xacro:property name="head_size_z" value="0.217" />
+	<xacro:property name="camara_frame_offset" value="0.021" />
+	<xacro:property name="f10_camara_offset_x" value="0.0075" />
+	<xacro:property name="f10_camara_offset_y" value="0.055" />
+	<xacro:property name="f10_camara_offset_z" value="0.015" />
+	<xacro:property name="f10_optical_offset" value="0.0145" />
+	<xacro:property name="xtion_camara_offset_x" value="0.041" />
+	<xacro:property name="xtion_camara_offset_y" value="0.0" />
+	<xacro:property name="xtion_camara_offset_z" value="0.065" />
+	<xacro:property name="head_joint_damping" value="0.0" />
+	<xacro:property name="head_joint_friction" value="0.0" />
+	<xacro:property name="head_joint_effort_limit" value="100.0" />
+	<xacro:property name="head_joint_velocity_limit" value="100.0" />
+	<xacro:property name="head_pan_joint_upper_limit" value="${M_PI/2}" />
+	<xacro:property name="head_pan_joint_lower_limit" value="${reverse*M_PI/2}" />
+	<xacro:property name="head_tilt_joint_upper_limit" value="${M_PI/2}" />
+	<xacro:property name="head_tilt_joint_lower_limit" value="${reverse*M_PI/2}" />
+	<!-- Define the head -->
+	<xacro:macro name="head_model" params="parent name color *origin">
+	<!-- BASE HEAD -->
+		<joint name="${name}_frame_joint" type="fixed">
+			<xacro:insert_block name="origin" />
+			<parent link="${parent}_link"/>
+			<child link="${name}_frame_link"/>
+		</joint>
+		<link name="${name}_frame_link">
+		  <visual>
+			<origin xyz="0 0 0" rpy="0 0 0" />
+			<geometry>
+			  <mesh filename = "package://crom2_description/meshes/CROM2_pantilt_1.STL"/>
+			</geometry>
+			<material name="Blue" />
+		  </visual>
+		  <collision>
+			<origin xyz="0 0 0" rpy="0 0 0" />
+			<geometry>
+			  <mesh filename = "package://crom2_description/meshes/CROM2_pantilt_1.dae" />
+			</geometry>
+		  </collision>
+		</link>
+	<!-- PAN HEAD -->
+		<joint name="${name}_pan_motor_joint" type="fixed">
+			<origin xyz="0 0 0" rpy="0 0 0" />
+			<parent link="${name}_frame_link"/>
+			<child link="${name}_pan_motor_link"/>
+		</joint>
+		<link name="${name}_pan_motor_link">
+		  <visual>
+			<origin xyz="0 0 0" rpy="0 0 0" />
+			<geometry>
+			  <mesh filename = "package://crom2_description/meshes/dynamixel_L42.STL" />
+			</geometry>
+			<material name="Black" />
+		  </visual>
+		  <collision>
+			<origin xyz="0 0 0" rpy="0 0 0" />
+			<geometry>
+			  <mesh filename = "package://crom2_description/meshes/dynamixel_L42.dae" />
+			</geometry>
+		  </collision>
+		</link>
+		<joint name="${name}_pan_joint" type="revolute">
+		  <origin xyz="0 0 ${head_pan_joint_offset_z}" rpy="0 0 0" />
+		  <parent link="${name}_pan_motor_link"/>
+		  <child link="${name}_pan_link"/>
+		  <axis xyz="0 0 1" />
+		  <limit effort="${head_joint_effort_limit}" velocity="${head_joint_velocity_limit}" upper="${head_tilt_joint_upper_limit}" lower="${head_tilt_joint_lower_limit}"/>
+		  <joint_properties damping="${head_joint_damping}" friction="{head_joint_friction}"/>
+		</joint>
+		<link name="${name}_pan_link">
+		  <visual>
+			<origin xyz="0 0 0" rpy="0 0 0" />
+			<geometry>
+			  <mesh filename = "package://crom2_description/meshes/CROM2_pantilt_2.STL" />
+			</geometry>
+			<material name="Blue" />
+		  </visual>
+		  <collision>
+			<origin xyz="0 0 0" rpy="0 0 0" />
+			<geometry>
+			  <mesh filename = "package://crom2_description/meshes/CROM2_pantilt_2.dae" />
+			</geometry>
+		  </collision>
+		</link>
+	<!-- TILT HEAD -->
+		<joint name="${name}_tilt_joint" type="revolute">
+		  <origin xyz="0 0 0" rpy="${reverse*M_PI/2} 0 0" />
+		  <parent link="${name}_pan_link"/>
+		  <child link="${name}_tilt_link"/>
+		  <axis xyz="0 0 -1" />
+		  <limit effort="${head_joint_effort_limit}" velocity="${head_joint_velocity_limit}" upper="${head_tilt_joint_upper_limit}" lower="${head_tilt_joint_lower_limit}"/>
+		  <joint_properties damping="${head_joint_damping}" friction="{head_joint_friction}"/>
+		</joint>
+		<link name="${name}_tilt_link">
+			<visual>
+			<origin xyz="0 0 ${reverse*head_tilt_servo_offset}" rpy="0 0 0" />
+			<geometry>
+			  <mesh filename = "package://crom2_description/meshes/dynamixel_L42.STL" />
+			</geometry>
+			<material name="Black" />
+		  </visual>
+		  <collision>
+			<origin xyz="0 0 ${head_tilt_servo_offset}" rpy="0 0 0" />
+			<geometry>
+			  <mesh filename = "package://crom2_description/meshes/dynamixel_L42.dae" />
+			</geometry>
+		  </collision>
+		</link>
+		<joint name="${name}_tilt_motor_joint" type="fixed">
+		  <origin xyz="0 0 0" rpy="0 0 0" />
+		  <parent link="${name}_pan_link"/>
+		  <child link="${name}_tilt_motor_link"/>
+		</joint>
+		<link name="${name}_tilt_motor_link">
+		  <visual>
+			<origin xyz="0 ${reverse*head_tilt_servo_offset} 0" rpy="0 0 0" />
+			<geometry>
+			  <mesh filename = "package://crom2_description/meshes/CROM2_pantilt_3.STL" />
+			</geometry>
+			<material name="Grey" />
+		  </visual>
+		  <collision>
+			<origin xyz="0 ${head_tilt_servo_offset} 0" rpy="0 0 0" />
+			<geometry>
+			  <mesh filename = "package://crom2_description/meshes/CROM2_pantilt_3.dae" />
+			</geometry>
+		  </collision>
+		</link>
+	<!-- CAMERA HEAD -->
+		<joint name="${name}_camera_frame_joint" type="fixed">
+		  <origin xyz="0 ${reverse*camara_frame_offset} 0" rpy="${M_PI/2}  0 0" />
+		  <parent link="${name}_tilt_link"/>
+		  <child link="${name}_camera_frame"/>
+		</joint>
+		<link name="${name}_camera_frame">
+		  <visual>
+			<origin xyz="0 0 0" rpy="0 0 0" />
+			<geometry>
+			  <mesh filename = "package://crom2_description/meshes/CROM2_pantilt_4.STL" />
+			</geometry>
+			<material name="Blue" />
+		  </visual>
+		  <collision>
+			<origin xyz="0 0 0" rpy="0 0 0" />
+			<geometry>
+			  <mesh filename = "package://crom2_description/meshes/CROM2_pantilt_4.dae" />
+			</geometry>
+		  </collision>
+		</link>
+	<!-- RIGHT CAMERA F10-->
+		<joint name="${name}_f10_camera_right_joint" type="fixed">
+		  <origin xyz="${f10_camara_offset_x} ${reverse*f10_camara_offset_y} ${f10_camara_offset_z}" rpy="0 0 0" />
+		  <parent link="${name}_camera_frame"/>
+		  <child link="${name}_f10_camera_right_frame"/>
+		</joint>
+		<link name="${name}_f10_camera_right_frame">
+		  <inertial>
+			<mass value="0.01" />
+			<origin xyz="0 0 0" />
+			<inertia  ixx="0.059" ixy="0.0"  ixz="0.0"  iyy="0.055"  iyz="0.0"  izz="0.059" />
+		  </inertial>
+		  <visual>
+			<origin xyz="0 0 0" rpy="0 0 0" />
+			<geometry>
+			  <mesh filename = "package://crom2_description/meshes/FL2-010-R0-camera.STL" />
+			</geometry>
+			<material name="Black" />
+		  </visual>
+		  <collision>
+			<origin xyz="0 0 0" rpy="0 0 0" />
+			<geometry>
+			  <mesh filename = "package://crom2_description/meshes/FL2-010-R0-camera.dae" />
+			</geometry>
+		  </collision>
+		</link>
+		<joint name="${name}_f10_camera_right_optical_joint" type="fixed">
+		  <origin xyz="0.0 0.0 ${f10_optical_offset}" rpy="${M_PI/2} 0 ${M_PI/2}" />
+		  <parent link="${name}_f10_camera_right_frame"/>
+		  <child link="${name}_f10_camera_right_optical_frame"/>
+		</joint>
+		<link name="${name}_f10_camera_right_optical_frame">
+		</link>
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
File: crom2_description/urdf/model/crom2_trunk.urdf.xacro (robot description, xacro)
@@ -1,11 +1,11 @@
 <?xml version="1.0"?>
 <robot name="trunk" xmlns:xacro="http://ros.org/wiki/xacro">
+  <xacro:include filename="$(find crom2_description)/urdf/gazebo/crom2_trunk.gazebo.xacro" />
   <!-- Define a number of dimensions using properties -->
   <property name="trunk_size_x" value="0.45" />
   <property name="trunk_size_y" value="0.284" />
   <property name="trunk_size_z" value="0.545" />
-  <property name="pi_2" value="1.57079" />
   <!-- Define the trunk -->
-  <macro name="trunk" params="parent name color *origin">
+  <xacro:macro name="trunk_model" params="parent name color *origin">
     <joint name="${name}_joint" type="revolute">
 		<xacro:insert_block name="origin" />
@@ -13,5 +13,5 @@
 		<child link="${name}_link" />
 		<axis xyz="0 0 1" />
-		<limit effort="1.5" velocity="1.0" lower="-${pi_2}" upper="${pi_2}" />
+		<limit effort="1.5" velocity="1.0" lower="${reverse*M_PI/2}" upper="${M_PI/2}" />
 	</joint>
 	<link name="${name}_link">
@@ -24,5 +24,4 @@
         <origin xyz="0 0 0" rpy="0 0 0" />
         <geometry>
-          <!--box size="${torso_size_x} ${torso_size_y} ${torso_size_z}" /-->
           <mesh filename = "package://crom2_description/meshes/CROM2_trunk.STL"/>
         </geometry>
@@ -32,9 +31,10 @@
         <origin xyz="0 0 0" rpy="0 0 0" />
         <geometry>
-			<mesh filename = "package://crom2_description/meshes/CROM2_trunk.dae"/>
-          <!--box size="${trunk_size_x} ${trunk_size_y} ${trunk_size_z}" /-->
+		  <mesh filename = "package://crom2_description/meshes/CROM2_trunk.dae"/>
         </geometry>
       </collision>
     </link>
-  </macro>
+    <!--Add trunk_gazebo macro -->
+	<trunk_gazebo name="${name}" />
+  </xacro:macro>
 </robot>

File: crom2_description/urdf/transmission/crom2_head.transmission.xacro (robot description, xacro)
@@ -1,106 +1,22 @@
 <?xml version="1.0"?>
 <robot xmlns:xacro="http://ros.org/wiki/xacro">
-	<xacro:macro name="head_gazebo" params="name">
-		<gazebo reference="${name}_start_link">
-			<fdir1 value="1 0 0"/>
-			<maxVel>2.0</maxVel>
-			<material>Gazebo/Grey</material>
-			<turnGravityOff>false</turnGravityOff>
-		</gazebo>
-		<gazebo reference="${name}_pan_link">
-			<fdir1 value="1 0 0"/>
-			<maxVel>2.0</maxVel>
-			<material>Gazebo/Grey</material>
-			<turnGravityOff>false</turnGravityOff>
-		</gazebo>
-		<gazebo reference="${name}_tilt_link">
-			<fdir1 value="1 0 0"/>
-			<maxVel>2.0</maxVel>
-			<material>Gazebo/Grey</material>
-			<turnGravityOff>false</turnGravityOff>
-		</gazebo>
-		<gazebo reference="${name}_camera_structure_link">
-			<material>Gazebo/FlatBlack</material>
-		</gazebo>
-	   <!-- camera_head_left_link -->
-	  <gazebo reference="${name}_camera_left_link">
-		<sensor type="camera" name="camera_head_left">
-		  <update_rate>30.0</update_rate>
-		  <camera name="camera_head_left">
-			<horizontal_fov>1.3962634</horizontal_fov>
-			<image>
-			  <width>800</width>
-			  <height>800</height>
-			  <format>R8G8B8</format>
-			</image>
-			<clip>
-			  <near>0.02</near>
-			  <far>300</far>
-			</clip>
-			<noise>
-			  <type>gaussian</type>
-			  <!-- Noise is sampled independently per pixel on each frame.
-				   That pixel's noise value is added to each of its color
-				   channels, which at that point lie in the range [0,1]. -->
-			  <mean>0.0</mean>
-			  <stddev>0.007</stddev>
-			</noise>
-		  </camera>
-		  <plugin name="camera_controller" filename="libgazebo_ros_camera.so">
-			<alwaysOn>true</alwaysOn>
-			<updateRate>0.0</updateRate>
-			<cameraName>crom/camera_head_left</cameraName>
-			<imageTopicName>image_raw</imageTopicName>
-			<cameraInfoTopicName>camera_head_left_info</cameraInfoTopicName>
-			<frameName>camera_head_left_link</frameName>
-			<hackBaseline>0.07</hackBaseline>
-			<distortionK1>0.0</distortionK1>
-			<distortionK2>0.0</distortionK2>
-			<distortionK3>0.0</distortionK3>
-			<distortionT1>0.0</distortionT1>
-			<distortionT2>0.0</distortionT2>
-		  </plugin>
-		</sensor>
-	  </gazebo>
-		<!-- camera_head_right_link -->
-	  <gazebo reference="${name}_camera_right_link">
-		<sensor type="camera" name="camera_head_right">
-		  <update_rate>30.0</update_rate>
-		  <camera name="camera_head_right">
-			<horizontal_fov>1.3962634</horizontal_fov>
-			<image>
-			  <width>800</width>
-			  <height>800</height>
-			  <format>R8G8B8</format>
-			</image>
-			<clip>
-			  <near>0.02</near>
-			  <far>300</far>
-			</clip>
-			<noise>
-			  <type>gaussian</type>
-			  <!-- Noise is sampled independently per pixel on each frame.
-				   That pixel's noise value is added to each of its color
-				   channels, which at that point lie in the range [0,1]. -->
-			  <mean>0.0</mean>
-			  <stddev>0.007</stddev>
-			</noise>
-		  </camera>
-		  <plugin name="camera_controller" filename="libgazebo_ros_camera.so">
-			<alwaysOn>true</alwaysOn>
-			<updateRate>0.0</updateRate>
-			<cameraName>crom/camera_head_right</cameraName>
-			<imageTopicName>image_raw</imageTopicName>
-			<cameraInfoTopicName>camera_head_right_info</cameraInfoTopicName>
-			<frameName>camera_hand_right_link</frameName>
-			<hackBaseline>0.07</hackBaseline>
-			<distortionK1>0.0</distortionK1>
-			<distortionK2>0.0</distortionK2>
-			<distortionK3>0.0</distortionK3>
-			<distortionT1>0.0</distortionT1>
-			<distortionT2>0.0</distortionT2>
-		  </plugin>
-		</sensor>
-	  </gazebo>
+	<xacro:macro name="head_transmission" params="name">
+		<xacro:property name="head_mechanical_reduction" value="1.0" />
+		<transmission name="${name}_joint_pan_transmission">
+			 <type>transmission_interface/SimpleTransmission</type>
+			 <joint name="${name}_pan_joint" />
+			 <actuator name="${name}_pan_motor">
+			   <hardwareInterface>PositionJointInterface</hardwareInterface>
+			   <mechanicalReduction>${head_mechanical_reduction}</mechanicalReduction>
+			 </actuator>
+		</transmission>
+		<transmission name="${name}_joint_tilt_transmisssion">
+			 <type>transmission_interface/SimpleTransmission</type>
+			 <joint name="${name}_tilt_joint" />
+			 <actuator name="${name}_tilt_motor">
+			   <hardwareInterface>PositionJointInterface</hardwareInterface>
+			   <mechanicalReduction>${head_mechanical_reduction}</mechanicalReduction>
+			 </actuator>
+		</transmission>
   </xacro:macro>
 </robot>
