Commit message: Solved: single ros_control

File: crom2_description/robots/crom2.gazebo.xacro (robot description, xacro)
@@ -4,5 +4,5 @@
 	  <gazebo>
 		<plugin name="gazebo_ros_control" filename="libgazebo_ros_control.so">
-			<robotNamespace>/crom2</robotNamespace>
+			<robotNamespace>/crom2/</robotNamespace>
 			<controlPeriod>0.001</controlPeriod>
 			<robotSimType>gazebo_ros_control/DefaultRobotHWSim</robotSimType>

File: crom2_description/robots/crom2_ur10.urdf.xacro (robot description, xacro)
@@ -2,7 +2,7 @@
 <robot name="crom2_robot" xmlns:xacro="http://ros.org/wiki/xacro">
    <!-- Define a offsets using properties -->
-   <property name="torso_offset_x" value="0.0" />
-   <property name="torso_offset_y" value="0.0" />
-   <property name="torso_offset_z" value="0.0" />
+   <property name="base_offset_x" value="0.0" />
+   <property name="base_offset_y" value="0.0" />
+   <property name="base_offset_z" value="0.0" />
    <property name="trunk_offset_x" value="0.0" />
    <property name="trunk_offset_y" value="0.0" />
@@ -11,29 +11,35 @@
    <property name="head_offset_y" value="0.0" />
    <property name="head_offset_z" value="0.545" />
-   <property name="pi_2" value="1.57079" />
+   <property name="reverse" value="-1.0" />
+   <property name="M_PI" value="3.1415926535897931" />
    <!-- Include all component files -->
-   <xacro:include filename="$(find crom2_description)/urdf/materials.urdf.xacro" />
-   <xacro:include filename="$(find crom2_description)/urdf/crom2_base.urdf.xacro" />
-   <xacro:include filename="$(find crom2_description)/urdf/crom2_trunk.urdf.xacro" />
-   <xacro:include filename="$(find crom2_description)/urdf/crom2_head.urdf.xacro" />
-   <xacro:include filename="$(find ur_description)/urdf/common.gazebo.xacro" />
+   <xacro:include filename="$(find crom2_description)/urdf/material/materials.urdf.xacro" />
+   <xacro:include filename="$(find crom2_description)/urdf/model/crom2_base.urdf.xacro" />
+   <xacro:include filename="$(find crom2_description)/urdf/model/crom2_trunk.urdf.xacro" />
+   <xacro:include filename="$(find crom2_description)/urdf/model/crom2_head.urdf.xacro" />
+   <xacro:include filename="$(find crom2_description)/robots/crom2.gazebo.xacro" />
+   <!-- Include arm component files -->
    <xacro:include filename="$(find ur_description)/urdf/ur10.urdf.xacro" />
   <link name="base_footprint">
   </link>
    <!-- Add the base -->
-   <base name="base" color="Blue" parent="base_footprint"/>
+   <base_model name="base" parent="base_footprint" color="Blue">
+	    <origin xyz="${base_offset_x} ${base_offset_y} ${base_offset_z}" rpy="0 0 0" />
+   </base_model>
    <!-- Attach the trunk -->
-   <trunk name="waist" parent="base" color="Blue">
+   <trunk_model name="waist" parent="base" color="Blue">
       <origin xyz="${trunk_offset_x} ${trunk_offset_y} ${trunk_offset_z}" rpy="0 0 0" />
-   </trunk>
+   </trunk_model>
    <!-- Attach the head -->
-   <head name="head" parent="waist" color="Blue">
+   <head_model name="head" parent="waist" color="Blue">
       <origin xyz="${head_offset_x} ${head_offset_y} ${head_offset_z}" rpy="0 0 0" />
-   </head>
-    <!-- arm -->
+   </head_model>
+   <!--IMPORTANT Add robot gazebo macro --> <!-- Add ros control to model -->
+   <crom2_gazebo />
+   <!-- Attach arms -->
    <joint name="right_arm_joint" type="fixed">
 		<parent link="waist_link" />
 		<child link = "right_arm_base_link" />
-		<origin xyz="0.0 -0.225 0.345" rpy="0 ${-pi_2} ${pi_2}" />
+		<origin xyz="0.0 -0.225 0.345" rpy="0 ${reverse*M_PI/2} ${M_PI/2}" />
    </joint>
    <xacro:ur10_robot prefix="right_arm_" joint_limited="true"/>
@@ -41,5 +47,5 @@
 		<parent link="waist_link" />
 		<child link = "left_arm_base_link" />
-		<origin xyz="0.0 0.225 0.345" rpy="0 -${pi_2} -${pi_2}" />
+		<origin xyz="0.0 0.225 0.345" rpy="0 ${reverse*M_PI/2} ${reverse*M_PI/2}" />
    </joint>
    <xacro:ur10_robot prefix="left_arm_" joint_limited="true"/>

File: crom2_description/robots/crom2_ur10_no_limits.urdf.xacro (robot description, xacro)
@@ -13,9 +13,9 @@
    <property name="pi_2" value="1.57079" />
    <!-- Include all component files -->
-   <xacro:include filename="$(find crom2_description)/urdf/materials.urdf.xacro" />
-   <xacro:include filename="$(find crom2_description)/urdf/crom2_base.urdf.xacro" />
-   <xacro:include filename="$(find crom2_description)/urdf/crom2_trunk.urdf.xacro" />
-   <xacro:include filename="$(find crom2_description)/urdf/crom2_head.urdf.xacro" />
-   <xacro:include filename="$(find ur_description)/urdf/common.gazebo.xacro" />
+   <xacro:include filename="$(find crom2_description)/urdf/material/materials.urdf.xacro" />
+   <xacro:include filename="$(find crom2_description)/urdf/model/crom2_base.urdf.xacro" />
+   <xacro:include filename="$(find crom2_description)/urdf/model/crom2_trunk.urdf.xacro" />
+   <xacro:include filename="$(find crom2_description)/urdf/model/crom2_head.urdf.xacro" />
+   <!--xacro:include filename="$(find ur_description)/urdf/common.gazebo.xacro" /-->
    <xacro:include filename="$(find ur_description)/urdf/ur10.urdf.xacro" />
   <link name="base_footprint">

File: crom2_description/urdf/model/crom2_head.urdf.xacro (robot description, xacro)
@@ -276,5 +276,5 @@
 			<origin xyz="0 0 0" rpy="0 0 0" />
 			<geometry>
-			  <mesh filename = "package://crom2_description/meshes/xtion_camera.dae " />
+			  <mesh filename = "package://crom2_description/meshes/xtion_camera.dae" />
 			</geometry>
 			<material name="Black" />
