Commit message: added some gazebo spects

File: crom2_description/robots/crom2_no_arms.urdf.xacro (robot description, xacro)
@@ -12,13 +12,13 @@
    <property name="head_offset_z" value="0.545" />
    <!-- Include all component files -->
-   <xacro:include filename="$(find crom2_description)/urdf/materials.urdf.xacro" />
-   <xacro:include filename="$(find crom2_description)/urdf/crom2_base.urdf.xacro" />
-   <xacro:include filename="$(find crom2_description)/urdf/crom2_trunk.urdf.xacro" />
-   <xacro:include filename="$(find crom2_description)/urdf/crom2_head.urdf.xacro" />
+   <xacro:include filename="$(find crom2_description)/urdf/material/materials.urdf.xacro" />
+   <xacro:include filename="$(find crom2_description)/urdf/model/crom2_base.urdf.xacro" />
+   <xacro:include filename="$(find crom2_description)/urdf/model/crom2_trunk.urdf.xacro" />
+   <xacro:include filename="$(find crom2_description)/urdf/model/crom2_head.urdf.xacro" />
    <!--xacro:include filename="$(find crom2_description)/urdf/crom2_head.urdf.xacro" /-->
   <link name="base_footprint">
   </link>
    <!-- Add the base -->
-   <base name="base" color="Blue" parent="base_footprint"/>
+   <base name="base" parent="base_footprint" color="Blue"/>
    <!-- Attach the trunk -->
    <trunk name="waist" parent="base" color="Blue">

File: crom2_description/urdf/model/crom2_base.urdf.xacro (robot description, xacro)
@@ -13,5 +13,5 @@
         <origin xyz="0 0 0" rpy="0 0 0" />
         <geometry>
-          <mesh filename = "package://crom2_description/meshes/CROM2_base.dae"/>
+          <mesh filename = "package://crom2_description/meshes/CROM2_base.STL"/>
         </geometry>
         <material name="${color}" />

File: crom2_description/urdf/model/crom2_head.urdf.xacro (robot description, xacro)
@@ -19,5 +19,5 @@
         <origin xyz="0 0 0" rpy="0 0 0" />
         <geometry>
-          <mesh filename = "package://crom2_description/meshes/CROM2_pantilt_1.dae"/>
+          <mesh filename = "package://crom2_description/meshes/CROM2_pantilt_1.STL"/>
         </geometry>
         <material name="Blue" />
@@ -39,5 +39,5 @@
         <origin xyz="0 0 0" rpy="0 0 0" />
         <geometry>
-          <mesh filename = "package://crom2_description/meshes/dynamixel_L42.dae" />
+          <mesh filename = "package://crom2_description/meshes/dynamixel_L42.STL" />
         </geometry>
         <material name="Black" />
@@ -61,5 +61,5 @@
         <origin xyz="0 0 0" rpy="0 0 0" />
         <geometry>
-          <mesh filename = "package://crom2_description/meshes/CROM2_pantilt_2.dae" />
+          <mesh filename = "package://crom2_description/meshes/CROM2_pantilt_2.STL" />
         </geometry>
         <material name="Blue" />
@@ -83,5 +83,5 @@
         <origin xyz="0 0 -0.027" rpy="0 0 0" />
         <geometry>
-          <mesh filename = "package://crom2_description/meshes/dynamixel_L42.dae" />
+          <mesh filename = "package://crom2_description/meshes/dynamixel_L42.STL" />
         </geometry>
         <material name="Black" />
@@ -103,5 +103,5 @@
         <origin xyz="0 -0.027 0" rpy="0 0 0" />
         <geometry>
-          <mesh filename = "package://crom2_description/meshes/CROM2_pantilt_3.dae" />
+          <mesh filename = "package://crom2_description/meshes/CROM2_pantilt_3.STL" />
         </geometry>
         <material name="Grey" />
@@ -123,5 +123,5 @@
         <origin xyz="0 0 0" rpy="0 0 0" />
         <geometry>
-          <mesh filename = "package://crom2_description/meshes/CROM2_pantilt_4.dae" />
+          <mesh filename = "package://crom2_description/meshes/CROM2_pantilt_4.STL" />
         </geometry>
         <material name="Blue" />
@@ -143,5 +143,5 @@
         <origin xyz="0 0 0" rpy="0 0 0" />
         <geometry>
-          <mesh filename = "package://crom2_description/meshes/FL2-010-R0-camera.dae" />
+          <mesh filename = "package://crom2_description/meshes/FL2-010-R0-camera.STL" />
         </geometry>
         <material name="Black" />
@@ -170,5 +170,5 @@
         <origin xyz="0 0 0" rpy="0 0 0" />
         <geometry>
-          <mesh filename = "package://crom2_description/meshes/FL2-010-R0-camera.dae" />
+          <mesh filename = "package://crom2_description/meshes/FL2-010-R0-camera.STL" />
         </geometry>
         <material name="Black" />
@@ -197,5 +197,5 @@
         <origin xyz="0 0 0" rpy="0 0 0" />
         <geometry>
-          <mesh filename = "package://crom2_description/meshes/xtion_camera.dae" />
+          <mesh filename = "package://crom2_description/meshes/xtion_camera.STL" />
         </geometry>
         <material name="Black" />

File: crom2_description/urdf/model/crom2_trunk.urdf.xacro (robot description, xacro)
@@ -5,7 +5,6 @@
   <property name="trunk_size_y" value="0.284" />
   <property name="trunk_size_z" value="0.545" />
-  <property name="mesh_scale" value="1" />
   <property name="pi_2" value="1.57079" />
-  <!-- Define the torso -->
+  <!-- Define the trunk -->
   <macro name="trunk" params="parent name color *origin">
     <joint name="${name}_joint" type="revolute">
@@ -17,9 +16,14 @@
 	</joint>
 	<link name="${name}_link">
+		<inertial>
+		  <mass value="22.07245" />
+		  <origin xyz="0 0 0" />
+		  <inertia  ixx="1259.328" ixy="-0.695"  ixz="15.497"  iyy="934.927"  iyz="-0.007"  izz="771.083" />
+		</inertial>
       <visual>
         <origin xyz="0 0 0" rpy="0 0 0" />
         <geometry>
           <!--box size="${torso_size_x} ${torso_size_y} ${torso_size_z}" /-->
-          <mesh filename = "package://crom2_description/meshes/CROM2_trunk.dae"/>
+          <mesh filename = "package://crom2_description/meshes/CROM2_trunk.STL"/>
         </geometry>
         <material name="${color}" />
