Commit message: added <inertial> tag to all links in model

File: crom2_description/robots/crom2_no_arms.urdf.xacro (robot description, xacro)
@@ -20,8 +20,9 @@
    <property name="head_offset_y" value="0.0" />
    <property name="head_offset_z" value="0.545" />
-  <link name="base_footprint">
-  </link>
+   <link name="base_footprint">
+   </link>
    <!-- Add the base -->
    <base_model name="base" parent="base_footprint" color="Blue">
+	    <origin xyz="${base_offset_x} ${base_offset_y} ${base_offset_z}" rpy="0 0 0" />
    </base_model>
    <!-- Attach the trunk -->

File: crom2_description/urdf/gazebo/crom2_head.gazebo.xacro (robot description, xacro)
@@ -2,113 +2,129 @@
 <robot xmlns:xacro="http://ros.org/wiki/xacro">
 	<xacro:macro name="head_gazebo" params="name">
-		<gazebo reference="$${name}_base_link">
-			<fdir1 value="1 0 0"/>
-			<maxVel>2.0</maxVel>
+		<gazebo reference="${name}_frame_link">
 			<material>Gazebo/Grey</material>
 			<turnGravityOff>false</turnGravityOff>
+			<selfCollide>true</selfCollide>
 		</gazebo>
 		<gazebo reference="${name}_pan_motor_link">
-			<fdir1 value="1 0 0"/>
-			<maxVel>2.0</maxVel>
+			<material>Gazebo/FlatBlack</material>
+			<turnGravityOff>false</turnGravityOff>
+			<selfCollide>true</selfCollide>
 		</gazebo>
 		<gazebo reference="${name}_pan_link">
-			<fdir1 value="1 0 0"/>
-			<maxVel>2.0</maxVel>
 			<material>Gazebo/Grey</material>
 			<turnGravityOff>false</turnGravityOff>
+			<selfCollide>true</selfCollide>
 		</gazebo>
 		<gazebo reference="${name}_tilt_motor_link">
-			<fdir1 value="1 0 0"/>
-			<maxVel>2.0</maxVel>
+			<material>Gazebo/FlatBlack</material>
+			<turnGravityOff>false</turnGravityOff>
+			<selfCollide>true</selfCollide>
 		</gazebo>
 		<gazebo reference="${name}_tilt_link">
-			<fdir1 value="1 0 0"/>
-			<material>Gazebo/FlatBlack</material>
 			<material>Gazebo/Grey</material>
 			<turnGravityOff>false</turnGravityOff>
+			<selfCollide>true</selfCollide>
 		</gazebo>
 		<gazebo reference="${name}_camera_frame">
+			<material>Gazebo/Grey</material>
+			<turnGravityOff>false</turnGravityOff>
+			<selfCollide>true</selfCollide>
+		</gazebo>
+		<gazebo reference="${name}_f10_camera_right_frame">
 			<material>Gazebo/FlatBlack</material>
+			<turnGravityOff>false</turnGravityOff>
+			<selfCollide>true</selfCollide>
 		</gazebo>
-	  <!-- camera_head_left_link -->
-	  <gazebo reference="${name}_f10_camera_left_optical_frame">
-		<sensor type="camera" name="${name}_f10_camera_left">
-		  <update_rate>30.0</update_rate>
-		  <camera name="${name}_f10_camera_left">
-			<horizontal_fov>1.3962634</horizontal_fov>
-			<image>
-			  <width>800</width>
-			  <height>800</height>
-			  <format>R8G8B8</format>
-			</image>
-			<clip>
-			  <near>0.02</near>
-			  <far>300</far>
-			</clip>
-			<noise>
-			  <type>gaussian</type>
-			  <!-- Noise is sampled independently per pixel on each frame.
-				   That pixel's noise value is added to each of its color
-				   channels, which at that point lie in the range [0,1]. -->
-			  <mean>0.0</mean>
-			  <stddev>0.007</stddev>
-			</noise>
-		  </camera>
-		  <plugin name="camera_controller" filename="libgazebo_ros_camera.so">
-			<alwaysOn>true</alwaysOn>
-			<updateRate>0.0</updateRate>
-			<cameraName>crom/camera_head_left</cameraName>
-			<imageTopicName>image_raw</imageTopicName>
-			<cameraInfoTopicName>camera_head_left_info</cameraInfoTopicName>
-			<frameName>camera_head_left_link</frameName>
-			<hackBaseline>0.07</hackBaseline>
-			<distortionK1>0.0</distortionK1>
-			<distortionK2>0.0</distortionK2>
-			<distortionK3>0.0</distortionK3>
-			<distortionT1>0.0</distortionT1>
-			<distortionT2>0.0</distortionT2>
-		  </plugin>
-		</sensor>
-	  </gazebo>
-	  <!-- camera_head_right_link -->
-	  <gazebo reference="{name}_f10_camera_right_optical_frame">
-		<sensor type="camera" name="${name}_f10_camera_right">
-		  <update_rate>30.0</update_rate>
-		  <camera name="${name}_f10_camera_right">
-			<horizontal_fov>1.3962634</horizontal_fov>
-			<image>
-			  <width>800</width>
-			  <height>800</height>
-			  <format>R8G8B8</format>
-			</image>
-			<clip>
-			  <near>0.02</near>
-			  <far>300</far>
-			</clip>
-			<noise>
-			  <type>gaussian</type>
-			  <!-- Noise is sampled independently per pixel on each frame.
-				   That pixel's noise value is added to each of its color
-				   channels, which at that point lie in the range [0,1]. -->
-			  <mean>0.0</mean>
-			  <stddev>0.007</stddev>
-			</noise>
-		  </camera>
-		  <plugin name="camera_controller" filename="libgazebo_ros_camera.so">
-			<alwaysOn>true</alwaysOn>
-			<updateRate>0.0</updateRate>
-			<cameraName>crom/camera_head_right</cameraName>
-			<imageTopicName>image_raw</imageTopicName>
-			<cameraInfoTopicName>camera_head_right_info</cameraInfoTopicName>
-			<frameName>camera_hand_right_link</frameName>
-			<hackBaseline>0.07</hackBaseline>
-			<distortionK1>0.0</distortionK1>
-			<distortionK2>0.0</distortionK2>
-			<distortionK3>0.0</distortionK3>
-			<distortionT1>0.0</distortionT1>
-			<distortionT2>0.0</distortionT2>
-		  </plugin>
-		</sensor>
-	  </gazebo>
+		<!-- camera_head_right_link -->
+		<gazebo reference="{name}_f10_camera_right_optical_frame">
+			<sensor type="camera" name="${name}_f10_camera_right">
+			  <update_rate>30.0</update_rate>
+			  <camera name="${name}_f10_camera_right">
+				<horizontal_fov>1.3962634</horizontal_fov>
+				<image>
+				  <width>800</width>
+				  <height>800</height>
+				  <format>R8G8B8</format>
+				</image>
+				<clip>
+				  <near>0.02</near>
+				  <far>300</far>
+				</clip>
+				<noise>
+				  <type>gaussian</type>
+				  <!-- Noise is sampled independently per pixel on each frame.
+					   That pixel's noise value is added to each of its color
+					   channels, which at that point lie in the range [0,1]. -->
+				  <mean>0.0</mean>
+				  <stddev>0.007</stddev>
+				</noise>
+			  </camera>
+			  <plugin name="camera_controller" filename="libgazebo_ros_camera.so">
+				<alwaysOn>true</alwaysOn>
+				<updateRate>0.0</updateRate>
+				<cameraName>crom/camera_head_right</cameraName>
+				<imageTopicName>image_raw</imageTopicName>
+				<cameraInfoTopicName>camera_head_right_info</cameraInfoTopicName>
+				<frameName>camera_hand_right_link</frameName>
+				<hackBaseline>0.07</hackBaseline>
+				<distortionK1>0.0</distortionK1>
+				<distortionK2>0.0</distortionK2>
+				<distortionK3>0.0</distortionK3>
+				<distortionT1>0.0</distortionT1>
+				<distortionT2>0.0</distortionT2>
+			  </plugin>
+			</sensor>
+		</gazebo>
+		<gazebo reference="${name}_f10_camera_left_frame">
+			<material>Gazebo/FlatBlack</material>
+			<turnGravityOff>false</turnGravityOff>
+			<selfCollide>true</selfCollide>
+		</gazebo>
+		<!-- camera_head_left_link -->
+		<gazebo reference="${name}_f10_camera_left_optical_frame">
+			<sensor type="camera" name="${name}_f10_camera_left">
+			  <update_rate>30.0</update_rate>
+			  <camera name="${name}_f10_camera_left">
+				<horizontal_fov>1.3962634</horizontal_fov>
+				<image>
+				  <width>800</width>
+				  <height>800</height>
+				  <format>R8G8B8</format>
+				</image>
+				<clip>
+				  <near>0.02</near>
+				  <far>300</far>
+				</clip>
+				<noise>
+				  <type>gaussian</type>
+				  <!-- Noise is sampled independently per pixel on each frame.
+					   That pixel's noise value is added to each of its color
+					   channels, which at that point lie in the range [0,1]. -->
+				  <mean>0.0</mean>
+				  <stddev>0.007</stddev>
+				</noise>
+			  </camera>
+			  <plugin name="camera_controller" filename="libgazebo_ros_camera.so">
+				<alwaysOn>true</alwaysOn>
+				<updateRate>0.0</updateRate>
+				<cameraName>crom/camera_head_left</cameraName>
+				<imageTopicName>image_raw</imageTopicName>
+				<cameraInfoTopicName>camera_head_left_info</cameraInfoTopicName>
+				<frameName>camera_head_left_link</frameName>
+				<hackBaseline>0.07</hackBaseline>
+				<distortionK1>0.0</distortionK1>
+				<distortionK2>0.0</distortionK2>
+				<distortionK3>0.0</distortionK3>
+				<distortionT1>0.0</distortionT1>
+				<distortionT2>0.0</distortionT2>
+			  </plugin>
+			</sensor>
+		</gazebo>
+		<gazebo reference="${name}_xtion_camera_frame">
+			<material>Gazebo/FlatBlack</material>
+			<turnGravityOff>false</turnGravityOff>
+			<selfCollide>true</selfCollide>
+		</gazebo>
   </xacro:macro>
 </robot>

File: crom2_description/urdf/model/crom2_base.urdf.xacro (robot description, xacro)
@@ -7,15 +7,24 @@
   <property name="base_size_z" value="1.078" />
   <!-- The base xacro macro -->
-  <xacro:macro name="base_model" params="name parent color">
+  <xacro:macro name="base_model" params="name parent color *origin">
     <joint name="${name}_joint" type="fixed">
-		<origin xyz="0 0 0" rpy="0 0 0" />
+		<xacro:insert_block name="origin" />
 		<parent link="${parent}"/>
 		<child link="${name}_link" />
 	</joint>
 	<link name="${name}_link">
+		 <!-- Inertial same to crom -->
+		<inertial>
+		  <mass value="800.0" />
+		  <origin xyz="0 0 0" />
+		  <inertia
+			ixx="3.737" ixy="0.008"  ixz="-0.144"
+			iyy="8.311"  iyz="-0.004"
+			izz="8.893" />
+		</inertial>
       <visual>
         <origin xyz="0 0 0" rpy="0 0 0" />
         <geometry>
-          <mesh filename = "package://crom2_description/meshes/CROM2_base.STL"/>
+          <mesh filename = "package://crom2_description/meshes/CROM2_base.dae"/>
         </geometry>
         <material name="${color}" />

File: crom2_description/urdf/model/crom2_head.urdf.xacro (robot description, xacro)
@@ -2,5 +2,5 @@
 <robot name="head" xmlns:xacro="http://ros.org/wiki/xacro">
 	<xacro:include filename="$(find crom2_description)/urdf/gazebo/crom2_head.gazebo.xacro" />
-	<!--xacro:include filename="$(find crom2_description)/urdf/transmission/crom2_head.transmission.xacro" /-->
+	<xacro:include filename="$(find crom2_description)/urdf/transmission/crom2_head.transmission.xacro" />
 	<!-- Define a number of dimensions using properties -->
 	<xacro:property name="head_pan_joint_offset_z" value="0.111" />
@@ -19,5 +19,5 @@
 	<xacro:property name="head_joint_damping" value="0.0" />
 	<xacro:property name="head_joint_friction" value="0.0" />
-	<xacro:property name="head_joint_effort_limit" value="100.0" />
+	<xacro:property name="head_joint_effort_limit" value="100.0" />_pan_joint
 	<xacro:property name="head_joint_velocity_limit" value="100.0" />
 	<xacro:property name="head_pan_joint_upper_limit" value="${M_PI/2}" />
@@ -37,5 +37,5 @@
 			<origin xyz="0 0 0" rpy="0 0 0" />
 			<geometry>
-			  <mesh filename = "package://crom2_description/meshes/CROM2_pantilt_1.STL"/>
+			  <mesh filename = "package://crom2_description/meshes/CROM2_pantilt_1.dae"/>
 			</geometry>
 			<material name="Blue" />
@@ -47,4 +47,12 @@
 			</geometry>
 		  </collision>
+		  <inertial>
+			<origin xyz="0 0 0" rpy="0 0 0" />
+			<mass value="1" />
+			<inertia
+			  ixx="1.0" ixy="0.0" ixz="0.0"
+			  iyy="1.0" iyz="0.0"
+			  izz="1.0" />
+		  </inertial>
 		</link>
 	<!-- PAN HEAD -->
@@ -58,14 +66,22 @@
 			<origin xyz="0 0 0" rpy="0 0 0" />
 			<geometry>
-			  <mesh filename = "package://crom2_description/meshes/dynamixel_L42.STL" />
-			</geometry>
-			<material name="Black" />
-		  </visual>
-		  <collision>
-			<origin xyz="0 0 0" rpy="0 0 0" />
-			<geometry>
 			  <mesh filename = "package://crom2_description/meshes/dynamixel_L42.dae" />
 			</geometry>
-		  </collision>
+			<material name="Black" />
+		  </visual>
+		  <collision>
+			<origin xyz="0 0 0" rpy="0 0 0" />
+			<geometry>
+			  <mesh filename = "package://crom2_description/meshes/dynamixel_L42.dae" />
+			</geometry>
+		  </collision>
+		  <inertial>
+			<origin xyz="0 0 0" rpy="0 0 0" />
+			<mass value="1" />
+			<inertia
+			  ixx="1.0" ixy="0.0" ixz="0.0"
+			  iyy="1.0" iyz="0.0"
+			  izz="1.0" />
+		  </inertial>
 		</link>
 		<joint name="${name}_pan_joint" type="revolute">
@@ -81,5 +97,5 @@
 			<origin xyz="0 0 0" rpy="0 0 0" />
 			<geometry>
-			  <mesh filename = "package://crom2_description/meshes/CROM2_pantilt_2.STL" />
+			  <mesh filename = "package://crom2_description/meshes/CROM2_pantilt_2.dae" />
 			</geometry>
 			<material name="Blue" />
@@ -91,4 +107,12 @@
 			</geometry>
 		  </collision>
+		  <inertial>
+			<origin xyz="0 0 0" rpy="0 0 0" />
+			<mass value="1" />
+			<inertia
+			  ixx="1.0" ixy="0.0" ixz="0.0"
+			  iyy="1.0" iyz="0.0"
+			  izz="1.0" />
+		  </inertial>
 		</link>
 	<!-- TILT HEAD -->
@@ -105,5 +129,5 @@
 			<origin xyz="0 0 ${reverse*head_tilt_servo_offset}" rpy="0 0 0" />
 			<geometry>
-			  <mesh filename = "package://crom2_description/meshes/dynamixel_L42.STL" />
+			  <mesh filename = "package://crom2_description/meshes/dynamixel_L42.dae" />
 			</geometry>
 			<material name="Black" />
@@ -115,4 +139,12 @@
 			</geometry>
 		  </collision>
+		  <inertial>
+			<origin xyz="0 0 ${head_tilt_servo_offset}" rpy="0 0 0" />
+			<mass value="1" />
+			<inertia
+			  ixx="1.0" ixy="0.0" ixz="0.0"
+			  iyy="1.0" iyz="0.0"
+			  izz="1.0" />
+		  </inertial>
 		</link>
 		<joint name="${name}_tilt_motor_joint" type="fixed">
@@ -125,5 +157,5 @@
 			<origin xyz="0 ${reverse*head_tilt_servo_offset} 0" rpy="0 0 0" />
 			<geometry>
-			  <mesh filename = "package://crom2_description/meshes/CROM2_pantilt_3.STL" />
+			  <mesh filename = "package://crom2_description/meshes/CROM2_pantilt_3.dae" />
 			</geometry>
 			<material name="Grey" />
@@ -146,5 +178,5 @@
 			<origin xyz="0 0 0" rpy="0 0 0" />
 			<geometry>
-			  <mesh filename = "package://crom2_description/meshes/CROM2_pantilt_4.STL" />
+			  <mesh filename = "package://crom2_description/meshes/CROM2_pantilt_4.dae" />
 			</geometry>
 			<material name="Blue" />
@@ -156,4 +188,12 @@
 			</geometry>
 		  </collision>
+		  <inertial>
+			<origin xyz="0 0 0" rpy="0 0 0" />
+			<mass value="1" />
+			<inertia
+			  ixx="1.0" ixy="0.0" ixz="0.0"
+			  iyy="1.0" iyz="0.0"
+			  izz="1.0" />
+		  </inertial>
 		</link>
 	<!-- RIGHT CAMERA F10-->
@@ -167,5 +207,8 @@
 			<mass value="0.01" />
 			<origin xyz="0 0 0" />
-			<inertia  ixx="0.059" ixy="0.0"  ixz="0.0"  iyy="0.055"  iyz="0.0"  izz="0.059" />
+			<inertia
+				ixx="0.059" ixy="0.0"  ixz="0.0"
+				iyy="0.055"  iyz="0.0"
+				izz="0.059" />
 		  </inertial>
 		  <visual>
@@ -205,5 +248,5 @@
 			<origin xyz="0 0 0" rpy="0 0 0" />
 			<geometry>
-			  <mesh filename = "package://crom2_description/meshes/FL2-010-R0-camera.STL" />
+			  <mesh filename = "package://crom2_description/meshes/FL2-010-R0-camera.dae" />
 			</geometry>
 			<material name="Black" />
@@ -233,5 +276,5 @@
 			<origin xyz="0 0 0" rpy="0 0 0" />
 			<geometry>
-			  <mesh filename = "package://crom2_description/meshes/xtion_camera.STL" />
+			  <mesh filename = "package://crom2_description/meshes/xtion_camera.dae " />
 			</geometry>
 			<material name="Black" />
@@ -243,9 +286,17 @@
 			</geometry>
 		  </collision>
-		</link>
+		  <inertial>
+			<origin xyz="0 0 0" rpy="0 0 0" />
+			<mass value="1" />
+			<inertia
+			  ixx="1.0" ixy="0.0" ixz="0.0"
+			  iyy="1.0" iyz="0.0"
+			  izz="1.0" />
+		  </inertial>
+		</link>
+		<!--Add head_transmission macro -->
+		<head_transmission name="${name}" />
 		<!--Add head_gazebo macro -->
 		<head_gazebo name="${name}" />
-		<!--Add head_transmission macro -->
-		<!--head_transmission name="${name}" /-->
 	</xacro:macro>
 </robot>

File: crom2_description/urdf/model/crom2_trunk.urdf.xacro (robot description, xacro)
@@ -2,4 +2,5 @@
 <robot name="trunk" xmlns:xacro="http://ros.org/wiki/xacro">
   <xacro:include filename="$(find crom2_description)/urdf/gazebo/crom2_trunk.gazebo.xacro" />
+  <xacro:include filename="$(find crom2_description)/urdf/transmission/crom2_trunk.transmission.xacro" />
   <!-- Define a number of dimensions using properties -->
   <property name="trunk_size_x" value="0.45" />
@@ -19,10 +20,13 @@
 		  <mass value="22.07245" />
 		  <origin xyz="0 0 0" />
-		  <inertia  ixx="1259.328" ixy="-0.695"  ixz="15.497"  iyy="934.927"  iyz="-0.007"  izz="771.083" />
+		  <inertia
+		  ixx="1259.328" ixy="-0.695"  ixz="15.497"
+		  iyy="934.927"  iyz="-0.007"
+		  izz="771.083"/>
 		</inertial>
       <visual>
         <origin xyz="0 0 0" rpy="0 0 0" />
         <geometry>
-          <mesh filename = "package://crom2_description/meshes/CROM2_trunk.STL"/>
+          <mesh filename = "package://crom2_description/meshes/CROM2_trunk.dae"/>
         </geometry>
         <material name="${color}" />
@@ -37,4 +41,6 @@
     <!--Add trunk_gazebo macro -->
 	<trunk_gazebo name="${name}" />
+	<!--Add trunk_gazebo macro -->
+	<trunk_transmission name="${name}" />
   </xacro:macro>
 </robot>

File: crom2_description/urdf/transmission/crom2_head.transmission.xacro (robot description, xacro)
@@ -1,9 +1,11 @@
 <?xml version="1.0"?>
 <robot xmlns:xacro="http://ros.org/wiki/xacro">
+	<xacro:property name="head_mechanical_reduction" value="1.0" />
 	<xacro:macro name="head_transmission" params="name">
-		<xacro:property name="head_mechanical_reduction" value="1.0" />
 		<transmission name="${name}_joint_pan_transmission">
 			 <type>transmission_interface/SimpleTransmission</type>
-			 <joint name="${name}_pan_joint" />
+			 <joint name="${name}_pan_joint">
+			   <hardwareInterface>PositionJointInterface</hardwareInterface>
+		     </joint>
 			 <actuator name="${name}_pan_motor">
 			   <hardwareInterface>PositionJointInterface</hardwareInterface>
@@ -11,7 +13,9 @@
 			 </actuator>
 		</transmission>
-		<transmission name="${name}_joint_tilt_transmisssion">
+		<transmission name="${name}_joint_tilt_transmission">
 			 <type>transmission_interface/SimpleTransmission</type>
-			 <joint name="${name}_tilt_joint" />
+			 <joint name="${name}_tilt_joint">
+				 <hardwareInterface>PositionJointInterface</hardwareInterface>
+		     </joint>
 			 <actuator name="${name}_tilt_motor">
 			   <hardwareInterface>PositionJointInterface</hardwareInterface>

File: crom2_description/urdf/transmission/crom2_trunk.transmission.xacro (robot description, xacro)
@@ -1,9 +1,11 @@
 <?xml version="1.0"?>
 <robot xmlns:xacro="http://ros.org/wiki/xacro">
+	<xacro:property name="trunk_mechanical_reduction" value="1.0" />
 	<xacro:macro name="trunk_transmission" params="name">
-		<xacro:property name="trunk_mechanical_reduction" value="1.0" />
 		<transmission name="${name}_joint_transmission">
 			 <type>transmission_interface/SimpleTransmission</type>
-			 <joint name="${name}_joint" />
+			 <joint name="${name}_joint">
+				 <hardwareInterface>PositionJointInterface</hardwareInterface>
+			 </joint>
 			 <actuator name="${name}_motor">
 			   <hardwareInterface>PositionJointInterface</hardwareInterface>
