Commit message: description: updating the head position (moved forward) and some fixes in the simulation

File: crom2_description/robots/crom2_no_arms.urdf.xacro (robot description, xacro)
@@ -17,5 +17,5 @@
    <property name="trunk_offset_y" value="0.0" />
    <property name="trunk_offset_z" value="1.078" />
-   <property name="head_offset_x" value="0.0" />
+   <property name="head_offset_x" value="0.093" />
    <property name="head_offset_y" value="0.0" />
    <property name="head_offset_z" value="0.545" />

File: crom2_description/robots/crom2_ur10.urdf.xacro (robot description, xacro)
@@ -8,5 +8,5 @@
    <property name="trunk_offset_y" value="0.0" />
    <property name="trunk_offset_z" value="1.078" />
-   <property name="head_offset_x" value="0.0" />
+   <property name="head_offset_x" value="0.093" />
    <property name="head_offset_y" value="0.0" />
    <property name="head_offset_z" value="0.545" />

File: crom2_description/urdf/gazebo/crom2_head.gazebo.xacro (robot description, xacro)
@@ -1,4 +1,5 @@
 <?xml version="1.0"?>
 <robot xmlns:xacro="http://ros.org/wiki/xacro">
+	<xacro:property name="M_PI" value="3.1415926535897931" />
 	<xacro:macro name="head_gazebo" params="name">
 		<gazebo reference="${name}_frame_link">
@@ -37,8 +38,7 @@
 			<selfCollide>true</selfCollide>
 		</gazebo>
-		<!-- camera_head_right_link -->
-		<gazebo reference="{name}_f10_camera_right_optical_frame">
+		<gazebo reference="${name}_f10_camera_right_frame">
 			<sensor type="camera" name="${name}_f10_camera_right">
-			  <update_rate>30.0</update_rate>
+			  <update_rate>7.0</update_rate>
 			  <camera name="${name}_f10_camera_right">
 				<horizontal_fov>1.3962634</horizontal_fov>
@@ -54,12 +54,9 @@
 				<noise>
 				  <type>gaussian</type>
-				  <!-- Noise is sampled independently per pixel on each frame.
-					   That pixel's noise value is added to each of its color
-					   channels, which at that point lie in the range [0,1]. -->
 				  <mean>0.0</mean>
 				  <stddev>0.007</stddev>
 				</noise>
 			  </camera>
-			  <plugin name="camera_controller" filename="libgazebo_ros_camera.so">
+			  <plugin name="camera_right_controller" filename="libgazebo_ros_camera.so">
 				<alwaysOn>true</alwaysOn>
 				<updateRate>0.0</updateRate>
@@ -67,5 +64,5 @@
 				<imageTopicName>image_raw</imageTopicName>
 				<cameraInfoTopicName>camera_head_right_info</cameraInfoTopicName>
-				<frameName>camera_hand_right_link</frameName>
+				<frameName>${name}_f10_camera_right_optical_frame</frameName>
 				<hackBaseline>0.07</hackBaseline>
 				<distortionK1>0.0</distortionK1>
@@ -82,8 +79,7 @@
 			<selfCollide>true</selfCollide>
 		</gazebo>
-		<!-- camera_head_left_link -->
-		<gazebo reference="${name}_f10_camera_left_optical_frame">
+		<gazebo reference="${name}_f10_camera_left_frame">
 			<sensor type="camera" name="${name}_f10_camera_left">
-			  <update_rate>30.0</update_rate>
+			  <update_rate>7.0</update_rate>
 			  <camera name="${name}_f10_camera_left">
 				<horizontal_fov>1.3962634</horizontal_fov>
@@ -99,12 +95,9 @@
 				<noise>
 				  <type>gaussian</type>
-				  <!-- Noise is sampled independently per pixel on each frame.
-					   That pixel's noise value is added to each of its color
-					   channels, which at that point lie in the range [0,1]. -->
 				  <mean>0.0</mean>
 				  <stddev>0.007</stddev>
 				</noise>
 			  </camera>
-			  <plugin name="camera_controller" filename="libgazebo_ros_camera.so">
+			  <plugin name="camera_left_controller" filename="libgazebo_ros_camera.so">
 				<alwaysOn>true</alwaysOn>
 				<updateRate>0.0</updateRate>
@@ -112,5 +105,5 @@
 				<imageTopicName>image_raw</imageTopicName>
 				<cameraInfoTopicName>camera_head_left_info</cameraInfoTopicName>
-				<frameName>camera_head_left_link</frameName>
+				<frameName>${name}_f10_camera_left_optical_frame</frameName>
 				<hackBaseline>0.07</hackBaseline>
 				<distortionK1>0.0</distortionK1>
@@ -127,4 +120,40 @@
 			<selfCollide>true</selfCollide>
 		</gazebo>
+		<gazebo reference="${name}_xtion_camera_depth_frame">
+		  <sensor type="depth" name="${name}_xtion_camera_depth_sensor">
+			<always_on>true</always_on>
+			<update_rate>20.0</update_rate>
+			<camera>
+			  <horizontal_fov>${60.0*M_PI/180.0}</horizontal_fov>
+			  <image>
+				<format>R8G8B8</format>
+				<width>640</width>
+				<height>480</height>
+			  </image>
+			  <clip>
+				<near>0.05</near>
+				<far>3.5</far>
+			  </clip>
+			</camera>
+			<plugin name="camera_xtion_controller" filename="libgazebo_ros_openni_kinect.so">
+			  <cameraName>crom2/camera_xtion</cameraName>
+			  <alwaysOn>true</alwaysOn>
+			  <updateRate>15</updateRate>
+			  <imageTopicName>rgb/image_raw</imageTopicName>
+			  <depthImageTopicName>depth/image_raw</depthImageTopicName>
+			  <pointCloudTopicName>depth/points</pointCloudTopicName>
+			  <cameraInfoTopicName>rgb/camera_info</cameraInfoTopicName>
+			  <depthImageCameraInfoTopicName>depth/camera_info</depthImageCameraInfoTopicName>
+			  <frameName>${name}_xtion_camera_depth_optical_frame</frameName>
+			  <baseline>0.1</baseline>
+			  <distortion_k1>0.0</distortion_k1>
+			  <distortion_k2>0.0</distortion_k2>
+			  <distortion_k3>0.0</distortion_k3>
+			  <distortion_t1>0.0</distortion_t1>
+			  <distortion_t2>0.0</distortion_t2>
+			  <pointCloudCutoff>0.4</pointCloudCutoff>
+			</plugin>
+		  </sensor>
+		</gazebo>
   </xacro:macro>
 </robot>

File: crom2_description/urdf/model/crom2_head.urdf.xacro (robot description, xacro)
@@ -39,5 +39,5 @@
 			<origin xyz="0 0 0" rpy="0 0 0" />
 			<geometry>
-			  <mesh filename = "package://crom2_description/meshes/CROM2_pantilt_1.dae"/>
+			  <mesh filename = "package://crom2_description/meshes/CROM2_pantilt_1_1.dae"/>
 			</geometry>
 			<material name="Blue" />
@@ -46,5 +46,5 @@
 			<origin xyz="0 0 0" rpy="0 0 0" />
 			<geometry>
-			  <mesh filename = "package://crom2_description/meshes/CROM2_pantilt_1.dae" />
+			  <mesh filename = "package://crom2_description/meshes/CROM2_pantilt_1_1.dae" />
 			</geometry>
 		  </collision>
