Commit message: description: Adding robot made up of crom torso + 2x ur10 arms

File: crom2_description/robots/crom2_ur10.urdf.xacro (robot description, xacro)
@@ -11,4 +11,5 @@
    <property name="head_offset_y" value="0.0" />
    <property name="head_offset_z" value="0.545" />
+   <property name="pi_2" value="1.57079" />
    <!-- Include all component files -->
    <xacro:include filename="$(find crom2_description)/urdf/materials.urdf.xacro" />
@@ -16,5 +17,6 @@
    <xacro:include filename="$(find crom2_description)/urdf/crom2_trunk.urdf.xacro" />
    <xacro:include filename="$(find crom2_description)/urdf/crom2_head.urdf.xacro" />
-   <!--xacro:include filename="$(find crom2_description)/urdf/crom2_head.urdf.xacro" /-->
+   <xacro:include filename="$(find ur_description)/urdf/common.gazebo.xacro" />
+   <xacro:include filename="$(find ur_description)/urdf/ur10.urdf.xacro" />
   <link name="base_footprint">
   </link>
@@ -29,3 +31,16 @@
       <origin xyz="${head_offset_x} ${head_offset_y} ${head_offset_z}" rpy="0 0 0" />
    </head>
+    <!-- arm -->
+   <joint name="right_arm_joint" type="fixed">
+		<parent link="waist_link" />
+		<child link = "right_arm_base_link" />
+		<origin xyz="0.0 -0.225 0.345" rpy="${pi_2} 0.0 0.0" />
+   </joint>
+   <xacro:ur10_robot prefix="right_arm_" joint_limited="false"/>
+   <joint name="left_arm_joint" type="fixed">
+		<parent link="waist_link" />
+		<child link = "left_arm_base_link" />
+		<origin xyz="0.0 0.225 0.345" rpy="-${pi_2} 0.0 0.0" />
+   </joint>
+   <xacro:ur10_robot prefix="left_arm_" joint_limited="false"/>
 </robot>

Commit message: Adding MoveIt config package for the Crom2 + 2 UR10 with joints range limited

File: crom2_description/robots/crom2_ur10.urdf.xacro (robot description, xacro)
@@ -35,12 +35,12 @@
 		<parent link="waist_link" />
 		<child link = "right_arm_base_link" />
-		<origin xyz="0.0 -0.225 0.345" rpy="${pi_2} 0.0 0.0" />
+		<origin xyz="0.0 -0.225 0.345" rpy="0 ${-pi_2} ${pi_2}" />
    </joint>
-   <xacro:ur10_robot prefix="right_arm_" joint_limited="false"/>
+   <xacro:ur10_robot prefix="right_arm_" joint_limited="true"/>
    <joint name="left_arm_joint" type="fixed">
 		<parent link="waist_link" />
 		<child link = "left_arm_base_link" />
-		<origin xyz="0.0 0.225 0.345" rpy="-${pi_2} 0.0 0.0" />
+		<origin xyz="0.0 0.225 0.345" rpy="0 -${pi_2} -${pi_2}" />
    </joint>
-   <xacro:ur10_robot prefix="left_arm_" joint_limited="false"/>
+   <xacro:ur10_robot prefix="left_arm_" joint_limited="true"/>
 </robot>

File: crom2_description/urdf/crom2_trunk.urdf.xacro (robot description, xacro)
@@ -6,4 +6,5 @@
   <property name="trunk_size_z" value="0.545" />
   <property name="mesh_scale" value="1" />
+  <property name="pi_2" value="1.57079" />
   <!-- Define the torso -->
   <macro name="trunk" params="parent name color *origin">
@@ -13,5 +14,5 @@
 		<child link="${name}_link" />
 		<axis xyz="0 0 1" />
-		<limit effort="1.5" velocity="6.178465545" lower="-1.58" upper="1.58" />
+		<limit effort="1.5" velocity="1.0" lower="-${pi_2}" upper="${pi_2}" />
 	</joint>
 	<link name="${name}_link">

Commit message: Adding arms to bringup, relocation right arm

File: crom2_description/robots/crom2_ur10.urdf.xacro (robot description, xacro)
@@ -41,5 +41,5 @@
 		<parent link="waist_link" />
 		<child link = "right_arm_base_link" />
-		<origin xyz="0.0 -0.225 0.345" rpy="0 ${reverse*M_PI/2} ${M_PI/2}" />
+		<origin xyz="0.0 -0.225 0.345" rpy="0 ${M_PI/2} ${-M_PI/2}" />
    </joint>
    <xacro:ur10_robot prefix="right_arm_" joint_limited="true"/>
