Commit message: Add dae files

File: crom2_description/urdf/crom2_base.urdf.xacro (robot description, xacro)
@@ -13,5 +13,5 @@
         <origin xyz="0 0 0" rpy="0 0 0" />
         <geometry>
-          <mesh filename = "package://crom2_description/meshes/CROM2_base.STL" scale="${mesh_scale} ${mesh_scale} ${mesh_scale}" />
+          <mesh filename = "package://crom2_description/meshes/CROM2_base.STL"/>
         </geometry>
         <material name="${color}" />

File: crom2_description/urdf/crom2_head.urdf.xacro (robot description, xacro)
@@ -18,5 +18,5 @@
         <origin xyz="0 0 0" rpy="0 0 0" />
         <geometry>
-          <mesh filename = "package://crom2_description/meshes/CROM2_pantilt_1.STL"/>
+          <mesh filename = "package://crom2_description/meshes/CROM2_pantilt_1.dae"/>
         </geometry>
         <material name="Blue" />
@@ -25,5 +25,5 @@
         <origin xyz="0 0 0" rpy="0 0 0" />
         <geometry>
-          <mesh filename = "package://crom2_description/meshes/CROM2_pantilt_1.STL" />
+          <mesh filename = "package://crom2_description/meshes/CROM2_pantilt_1.dae" />
         </geometry>
       </collision>
@@ -38,5 +38,5 @@
         <origin xyz="0 0 0" rpy="0 0 0" />
         <geometry>
-          <mesh filename = "package://crom2_description/meshes/dynamixel_L42.STL" />
+          <mesh filename = "package://crom2_description/meshes/dynamixel_L42.dae" />
         </geometry>
         <material name="Black" />
@@ -45,5 +45,5 @@
         <origin xyz="0 0 0" rpy="0 0 0" />
         <geometry>
-          <mesh filename = "package://crom2_description/meshes/dynamixel_L42.STL" />
+          <mesh filename = "package://crom2_description/meshes/dynamixel_L42.dae" />
         </geometry>
       </collision>
@@ -60,5 +60,5 @@
         <origin xyz="0 0 0" rpy="0 0 0" />
         <geometry>
-          <mesh filename = "package://crom2_description/meshes/CROM2_pantilt_2.STL" />
+          <mesh filename = "package://crom2_description/meshes/CROM2_pantilt_2.dae" />
         </geometry>
         <material name="Blue" />
@@ -67,5 +67,5 @@
         <origin xyz="0 0 0" rpy="0 0 0" />
         <geometry>
-          <mesh filename = "package://crom2_description/meshes/CROM2_pantilt_2.STL" />
+          <mesh filename = "package://crom2_description/meshes/CROM2_pantilt_2.dae" />
         </geometry>
       </collision>
@@ -82,5 +82,5 @@
         <origin xyz="0 0 -0.027" rpy="0 0 0" />
         <geometry>
-          <mesh filename = "package://crom2_description/meshes/dynamixel_L42.STL" />
+          <mesh filename = "package://crom2_description/meshes/dynamixel_L42.dae" />
         </geometry>
         <material name="Black" />
@@ -89,5 +89,5 @@
         <origin xyz="0 0 -0.027" rpy="0 0 0" />
         <geometry>
-          <mesh filename = "package://crom2_description/meshes/dynamixel_L42.STL" />
+          <mesh filename = "package://crom2_description/meshes/dynamixel_L42.dae" />
         </geometry>
       </collision>
@@ -102,5 +102,5 @@
         <origin xyz="0 -0.027 0" rpy="0 0 0" />
         <geometry>
-          <mesh filename = "package://crom2_description/meshes/CROM2_pantilt_3.STL" />
+          <mesh filename = "package://crom2_description/meshes/CROM2_pantilt_3.dae" />
         </geometry>
         <material name="Grey" />
@@ -109,5 +109,5 @@
         <origin xyz="0 -0.027 0" rpy="0 0 0" />
         <geometry>
-          <mesh filename = "package://crom2_description/meshes/CROM2_pantilt_3.STL" />
+          <mesh filename = "package://crom2_description/meshes/CROM2_pantilt_3.dae" />
         </geometry>
       </collision>
@@ -122,5 +122,5 @@
         <origin xyz="0 0 0" rpy="0 0 0" />
         <geometry>
-          <mesh filename = "package://crom2_description/meshes/CROM2_pantilt_4.STL" />
+          <mesh filename = "package://crom2_description/meshes/CROM2_pantilt_4.dae" />
         </geometry>
         <material name="Blue" />
@@ -129,5 +129,5 @@
         <origin xyz="0 0 0" rpy="0 0 0" />
         <geometry>
-          <mesh filename = "package://crom2_description/meshes/CROM2_pantilt_4.STL" />
+          <mesh filename = "package://crom2_description/meshes/CROM2_pantilt_4.dae" />
         </geometry>
       </collision>
@@ -142,5 +142,5 @@
         <origin xyz="0 0 0" rpy="0 0 0" />
         <geometry>
-          <mesh filename = "package://crom2_description/meshes/FL2-010-R0-camera.STL" />
+          <mesh filename = "package://crom2_description/meshes/FL2-010-R0-camera.dae" />
         </geometry>
         <material name="Black" />
@@ -149,5 +149,5 @@
         <origin xyz="0 0 0" rpy="0 0 0" />
         <geometry>
-          <mesh filename = "package://crom2_description/meshes/FL2-010-R0-camera.STL" />
+          <mesh filename = "package://crom2_description/meshes/FL2-010-R0-camera.dae" />
         </geometry>
       </collision>
@@ -162,5 +162,5 @@
         <origin xyz="0 0 0" rpy="0 0 0" />
         <geometry>
-          <mesh filename = "package://crom2_description/meshes/FL2-010-R0-camera.STL" />
+          <mesh filename = "package://crom2_description/meshes/FL2-010-R0-camera.dae" />
         </geometry>
         <material name="Black" />
@@ -169,5 +169,5 @@
         <origin xyz="0 0 0" rpy="0 0 0" />
         <geometry>
-          <mesh filename = "package://crom2_description/meshes/FL2-010-R0-camera.STL" />
+          <mesh filename = "package://crom2_description/meshes/FL2-010-R0-camera.dae" />
         </geometry>
       </collision>
@@ -182,5 +182,5 @@
         <origin xyz="0 0 0" rpy="0 0 0" />
         <geometry>
-          <mesh filename = "package://crom2_description/meshes/xtion_camera.STL" />
+          <mesh filename = "package://crom2_description/meshes/xtion_camera.dae" />
         </geometry>
         <material name="Black" />
@@ -189,5 +189,5 @@
         <origin xyz="0 0 0" rpy="0 0 0" />
         <geometry>
-          <mesh filename = "package://crom2_description/meshes/xtion_camera.STL" />
+          <mesh filename = "package://crom2_description/meshes/xtion_camera.dae" />
         </geometry>
       </collision>

File: crom2_description/urdf/crom2_trunk.urdf.xacro (robot description, xacro)
@@ -20,5 +20,5 @@
         <geometry>
           <!--box size="${torso_size_x} ${torso_size_y} ${torso_size_z}" /-->
-          <mesh filename = "package://crom2_description/meshes/CROM2_trunk.STL" scale="${mesh_scale} ${mesh_scale} ${mesh_scale}" />
+          <mesh filename = "package://crom2_description/meshes/CROM2_trunk.dae"/>
         </geometry>
         <material name="${color}" />

Commit message: description: replacing .stl of the base by .dae. Changing collision geometry of base and torso

File: crom2_description/urdf/crom2_base.urdf.xacro (robot description, xacro)
@@ -13,5 +13,5 @@
         <origin xyz="0 0 0" rpy="0 0 0" />
         <geometry>
-          <mesh filename = "package://crom2_description/meshes/CROM2_base.STL"/>
+          <mesh filename = "package://crom2_description/meshes/CROM2_base.dae"/>
         </geometry>
         <material name="${color}" />
@@ -20,5 +20,6 @@
         <origin xyz="0 0 0" rpy="0 0 0" />
         <geometry>
-          <box size="${base_size_x} ${base_size_y} ${base_size_z}" />
+          <!--box size="${base_size_x} ${base_size_y} ${base_size_z}" /-->
+           <mesh filename = "package://crom2_description/meshes/CROM2_base.dae"/>
         </geometry>
       </collision>

File: crom2_description/urdf/crom2_trunk.urdf.xacro (robot description, xacro)
@@ -27,5 +27,6 @@
         <origin xyz="0 0 0" rpy="0 0 0" />
         <geometry>
-          <box size="${trunk_size_x} ${trunk_size_y} ${trunk_size_z}" />
+			<mesh filename = "package://crom2_description/meshes/CROM2_trunk.dae"/>
+          <!--box size="${trunk_size_x} ${trunk_size_y} ${trunk_size_z}" /-->
         </geometry>
       </collision>
