Commit message: Adding package for the bringup

File: crom2_description/urdf/crom2_head.urdf.xacro (robot description, xacro)
@@ -75,5 +75,5 @@
       <parent link="${name}_pan_link"/>
       <child link="${name}_tilt_link"/>
-      <axis xyz="0 0 1" />
+      <axis xyz="0 0 -1" />
 	  <limit effort="1.5" velocity="6.178465545" lower="-1.57079" upper="1.57079" />
     </joint>

Commit message: Added pg optical frame

File: crom2_description/urdf/crom2_head.urdf.xacro (robot description, xacro)
@@ -7,4 +7,5 @@
   <property name="head_size_z" value="0.545" />
   <property name="mesh_scale" value="1" />
+  <property name="M_PI" value="3.1415926535897931" />
   <!-- Define the head -->
   <macro name="head" params="parent name color *origin">
@@ -116,7 +117,7 @@
       <origin xyz="0 -0.021 0" rpy="1.57079  0 0" />
       <parent link="${name}_tilt_link"/>
-      <child link="${name}_camera_frame_link"/>
-    </joint>
-    <link name="${name}_camera_frame_link">
+      <child link="${name}_camera_frame"/>
+    </joint>
+    <link name="${name}_camera_frame">
       <visual>
         <origin xyz="0 0 0" rpy="0 0 0" />
@@ -135,48 +136,62 @@
     <joint name="${name}_f10_camera_right_joint" type="fixed">
       <origin xyz="0.0075 -0.055 0.015" rpy="0 0 0" />
-      <parent link="${name}_camera_frame_link"/>
-      <child link="${name}_f10_camera_right_link"/>
-    </joint>
-    <link name="${name}_f10_camera_right_link">
-      <visual>
-        <origin xyz="0 0 0" rpy="0 0 0" />
-        <geometry>
-          <mesh filename = "package://crom2_description/meshes/FL2-010-R0-camera.dae" />
-        </geometry>
-        <material name="Black" />
-      </visual>
-      <collision>
-        <origin xyz="0 0 0" rpy="0 0 0" />
-        <geometry>
-          <mesh filename = "package://crom2_description/meshes/FL2-010-R0-camera.dae" />
-        </geometry>
-      </collision>
-    </link>
-      <joint name="${name}_f10_camera_left_joint" type="fixed">
+      <parent link="${name}_camera_frame"/>
+      <child link="${name}_f10_camera_right_frame"/>
+    </joint>
+    <link name="${name}_f10_camera_right_frame">
+      <visual>
+        <origin xyz="0 0 0" rpy="0 0 0" />
+        <geometry>
+          <mesh filename = "package://crom2_description/meshes/FL2-010-R0-camera.dae" />
+        </geometry>
+        <material name="Black" />
+      </visual>
+      <collision>
+        <origin xyz="0 0 0" rpy="0 0 0" />
+        <geometry>
+          <mesh filename = "package://crom2_description/meshes/FL2-010-R0-camera.dae" />
+        </geometry>
+      </collision>
+    </link>
+    <joint name="${name}_f10_camera_right_optical_joint" type="fixed">
+      <origin xyz="0.0 0.0 0.0145" rpy="${M_PI/2} 0 ${M_PI/2}" />
+      <parent link="${name}_f10_camera_right_frame"/>
+      <child link="${name}_f10_camera_right_optical_frame"/>
+    </joint>
+    <link name="${name}_f10_camera_right_optical_frame">
+    </link>
+    <joint name="${name}_f10_camera_left_joint" type="fixed">
       <origin xyz="0.0075 0.055 0.015" rpy="0 0 0" />
-      <parent link="${name}_camera_frame_link"/>
-      <child link="${name}_f10_camera_left_link"/>
-    </joint>
-    <link name="${name}_f10_camera_left_link">
-      <visual>
-        <origin xyz="0 0 0" rpy="0 0 0" />
-        <geometry>
-          <mesh filename = "package://crom2_description/meshes/FL2-010-R0-camera.dae" />
-        </geometry>
-        <material name="Black" />
-      </visual>
-      <collision>
-        <origin xyz="0 0 0" rpy="0 0 0" />
-        <geometry>
-          <mesh filename = "package://crom2_description/meshes/FL2-010-R0-camera.dae" />
-        </geometry>
-      </collision>
+      <parent link="${name}_camera_frame"/>
+      <child link="${name}_f10_camera_left_frame"/>
+    </joint>
+    <link name="${name}_f10_camera_left_frame">
+      <visual>
+        <origin xyz="0 0 0" rpy="0 0 0" />
+        <geometry>
+          <mesh filename = "package://crom2_description/meshes/FL2-010-R0-camera.dae" />
+        </geometry>
+        <material name="Black" />
+      </visual>
+      <collision>
+        <origin xyz="0 0 0" rpy="0 0 0" />
+        <geometry>
+          <mesh filename = "package://crom2_description/meshes/FL2-010-R0-camera.dae" />
+        </geometry>
+      </collision>
+    </link>
+    <joint name="${name}_f10_camera_left_optical_joint" type="fixed">
+      <origin xyz="0.0 0.0 0.0145" rpy="${M_PI/2} 0 ${M_PI/2}" />
+      <parent link="${name}_f10_camera_left_frame"/>
+      <child link="${name}_f10_camera_left_optical_frame"/>
+    </joint>
+    <link name="${name}_f10_camera_left_optical_frame">
     </link>
     <joint name="${name}_xtion_camera_joint" type="fixed">
       <origin xyz="0.041 0 0.065" rpy="0 0 0" />
-      <parent link="${name}_camera_frame_link"/>
-      <child link="${name}_xtion_camera_link"/>
-    </joint>
-    <link name="${name}_xtion_camera_link">
+      <parent link="${name}_camera_frame"/>
+      <child link="${name}_xtion_camera_frame"/>
+    </joint>
+    <link name="${name}_xtion_camera_frame">
       <visual>
         <origin xyz="0 0 0" rpy="0 0 0" />
