Commit message: Minor changes to base urdf

File: crom2_description/urdf/model/crom2_base.urdf.xacro (robot description, xacro)
@@ -14,14 +14,5 @@
 	</joint>
 	<link name="${name}_link">
-		 <!-- Inertial same to crom -->
-		<inertial>
-		  <mass value="800.0" />
-		  <origin xyz="0 0 0" />
-		  <inertia
-			ixx="3.737" ixy="0.008"  ixz="-0.144"
-			iyy="8.311"  iyz="-0.004"
-			izz="8.893" />
-		</inertial>
-      <visual>
+	  <visual>
         <origin xyz="0 0 0" rpy="0 0 0" />
         <geometry>
@@ -36,4 +27,13 @@
         </geometry>
       </collision>
+      <!-- Inertial same to crom -->
+		<inertial>
+		  <mass value="800.0" />
+		  <origin xyz="0 0 0" />
+		  <inertia
+			ixx="3.737" ixy="0.008"  ixz="-0.144"
+			iyy="8.311"  iyz="-0.004"
+			izz="8.893" />
+		</inertial>
     </link>
 	<!--Add base_gazebo macro -->
