Commit message: description: replacing .stl by .dae

File: crom2_description/urdf/model/crom2_head.urdf.xacro (robot description, xacro)
@@ -217,5 +217,5 @@
 			<origin xyz="0 0 0" rpy="0 0 0" />
 			<geometry>
-			  <mesh filename = "package://crom2_description/meshes/FL2-010-R0-camera.STL" />
+			  <mesh filename = "package://crom2_description/meshes/FL2-010-R0-camera.dae" />
 			</geometry>
 			<material name="Black" />

Commit message: description: setting tilt ranges between -1 and 1 rads

File: crom2_description/urdf/model/crom2_head.urdf.xacro (robot description, xacro)
@@ -23,6 +23,6 @@
 	<xacro:property name="head_pan_joint_upper_limit" value="${M_PI/2}" />
 	<xacro:property name="head_pan_joint_lower_limit" value="${reverse*M_PI/2}" />
-	<xacro:property name="head_tilt_joint_upper_limit" value="${M_PI/2}" />
-	<xacro:property name="head_tilt_joint_lower_limit" value="${reverse*M_PI/2}" />
+	<xacro:property name="head_tilt_joint_upper_limit" value="1.0" />
+	<xacro:property name="head_tilt_joint_lower_limit" value="-1.0" />
 	<xacro:property name="asus_xtion_pro_depth_rel_rgb_py" value="0.0270" />
 	<xacro:property name="asus_xtion_pro_cam_rel_rgb_py"   value="0.0220" />
