Commit message: color changes

File: crom2_description/urdf/gazebo/crom2_head.gazebo.xacro (robot description, xacro)
@@ -3,5 +3,5 @@
 	<xacro:macro name="head_gazebo" params="name">
 		<gazebo reference="${name}_frame_link">
-			<material>Gazebo/Grey</material>
+			<material>Gazebo/Blue</material>
 			<turnGravityOff>false</turnGravityOff>
 			<selfCollide>true</selfCollide>
@@ -13,5 +13,5 @@
 		</gazebo>
 		<gazebo reference="${name}_pan_link">
-			<material>Gazebo/Grey</material>
+			<material>Gazebo/Blue</material>
 			<turnGravityOff>false</turnGravityOff>
 			<selfCollide>true</selfCollide>
@@ -23,10 +23,10 @@
 		</gazebo>
 		<gazebo reference="${name}_tilt_link">
-			<material>Gazebo/Grey</material>
+			<material>Gazebo/FlatBlack</material>
 			<turnGravityOff>false</turnGravityOff>
 			<selfCollide>true</selfCollide>
 		</gazebo>
 		<gazebo reference="${name}_camera_frame">
-			<material>Gazebo/Grey</material>
+			<material>Gazebo/Blue</material>
 			<turnGravityOff>false</turnGravityOff>
 			<selfCollide>true</selfCollide>

Commit message: description: Setting rgbd frames for to work with openni2

File: crom2_description/urdf/gazebo/crom2_head.gazebo.xacro (robot description, xacro)
@@ -27,5 +27,5 @@
 			<selfCollide>true</selfCollide>
 		</gazebo>
-		<gazebo reference="${name}_camera_frame">
+		<gazebo reference="${name}_camera_link">
 			<material>Gazebo/Blue</material>
 			<turnGravityOff>false</turnGravityOff>
@@ -122,5 +122,5 @@
 			</sensor>
 		</gazebo>
-		<gazebo reference="${name}_xtion_camera_frame">
+		<gazebo reference="${name}_xtion_camera_link">
 			<material>Gazebo/FlatBlack</material>
 			<turnGravityOff>false</turnGravityOff>

File: crom2_description/urdf/model/crom2_head.urdf.xacro (robot description, xacro)
@@ -25,4 +25,6 @@
 	<xacro:property name="head_tilt_joint_upper_limit" value="${M_PI/2}" />
 	<xacro:property name="head_tilt_joint_lower_limit" value="${reverse*M_PI/2}" />
+	<xacro:property name="asus_xtion_pro_depth_rel_rgb_py" value="0.0270" />
+	<xacro:property name="asus_xtion_pro_cam_rel_rgb_py"   value="0.0220" />
 	<!-- Define the head -->
 	<xacro:macro name="head_model" params="parent name color *origin">
@@ -172,7 +174,7 @@
 		  <origin xyz="0 ${reverse*camara_frame_offset} 0" rpy="${M_PI/2}  0 0" />
 		  <parent link="${name}_tilt_link"/>
-		  <child link="${name}_camera_frame"/>
-		</joint>
-		<link name="${name}_camera_frame">
+		  <child link="${name}_camera_link"/>
+		</joint>
+		<link name="${name}_camera_link">
 		  <visual>
 			<origin xyz="0 0 0" rpy="0 0 0" />
@@ -200,5 +202,5 @@
 		<joint name="${name}_f10_camera_right_joint" type="fixed">
 		  <origin xyz="${f10_camara_offset_x} ${reverse*f10_camara_offset_y} ${f10_camara_offset_z}" rpy="0 0 0" />
-		  <parent link="${name}_camera_frame"/>
+		  <parent link="${name}_camera_link"/>
 		  <child link="${name}_f10_camera_right_frame"/>
 		</joint>
@@ -236,5 +238,5 @@
 		<joint name="${name}_f10_camera_left_joint" type="fixed">
 		  <origin xyz="${f10_camara_offset_x} ${f10_camara_offset_y} ${f10_camara_offset_z}" rpy="0 0 0" />
-		  <parent link="${name}_camera_frame"/>
+		  <parent link="${name}_camera_link"/>
 		  <child link="${name}_f10_camera_left_frame"/>
 		</joint>
@@ -266,11 +268,11 @@
 		<link name="${name}_f10_camera_left_optical_frame">
 		</link>
-	<!-- XTION CAMERA-->
+		<!-- XTION CAMERA-->
 		<joint name="${name}_xtion_camera_joint" type="fixed">
 		  <origin xyz="${xtion_camara_offset_x} ${xtion_camara_offset_y} ${xtion_camara_offset_z}" rpy="0 0 0" />
-		  <parent link="${name}_camera_frame"/>
-		  <child link="${name}_xtion_camera_frame"/>
-		</joint>
-		<link name="${name}_xtion_camera_frame">
+		  <parent link="${name}_camera_link"/>
+		  <child link="${name}_xtion_camera_link"/>
+		</joint>
+		<link name="${name}_xtion_camera_link">
 		  <visual>
 			<origin xyz="0 0 0" rpy="0 0 0" />
@@ -295,4 +297,29 @@
 		  </inertial>
 		</link>
+		<joint name="${name}_xtion_camera_rgb_joint" type="fixed">
+		  <origin xyz="0 ${asus_xtion_pro_cam_rel_rgb_py} 0"
+				  rpy="0 0 0"/>
+		  <parent link="${name}_xtion_camera_link"/>
+		  <child link="${name}_xtion_camera_rgb_frame" />
+		</joint>
+		<link name="${name}_xtion_camera_rgb_frame"/>
+		<joint name="${name}_xtion_camera_rgb_optical_joint" type="fixed">
+		  <origin xyz="0 0 0" rpy="${-M_PI/2} 0 ${-M_PI/2}" />
+		  <parent link="${name}_xtion_camera_rgb_frame" />
+		  <child link="${name}_xtion_camera_rgb_optical_frame" />
+		</joint>
+		<link name="${name}_xtion_camera_rgb_optical_frame"/>
+		<joint name="${name}_xtion_camera_depth_joint" type="fixed">
+		  <origin xyz="0 ${asus_xtion_pro_depth_rel_rgb_py} 0" rpy="0 0 0" />
+		  <parent link="${name}_xtion_camera_rgb_frame" />
+		  <child link="${name}_xtion_camera_depth_frame" />
+		</joint>
+		<link name="${name}_xtion_camera_depth_frame"/>
+		<joint name="${name}_xtion_camera_depth_optical_joint" type="fixed">
+		  <origin xyz="0 0 0" rpy="${-M_PI/2} 0 ${-M_PI/2}" />
+		  <parent link="${name}_xtion_camera_depth_frame" />
+		  <child link="${name}_xtion_camera_depth_optical_frame" />
+		</joint>
+		<link name="${name}_xtion_camera_depth_optical_frame"/>
 		<!--Add head_transmission macro -->
 		<head_transmission name="${name}" />
